Commit message: Fix joint issues

File: src/panther_description/urdf/chassis.urdf.xacro (robot description, xacro)
@@ -1,8 +1,8 @@
 <?xml version="1.0" encoding="utf-8"?>
 <robot xmlns:xacro="http://www.ros.org/wiki/xacro">
-  <!-- base_link defining macro -->
-  <xacro:macro name="base_link" params="props">
-    <link name="dummy"></link>
-    <link name="base_link">
+  <!-- chassis defining macro -->
+  <xacro:macro name="chassis" params="props">
+    <link name="base_link"></link>
+    <link name="chassis_link">
       <visual>
         <geometry>
@@ -30,7 +30,7 @@
       </inertial>
     </link>
-    <link name="cover">
+    <link name="cover_link">
       <inertial>
-        <mass value="0.00000000001" />
+        <mass value="0.0000001" />
         <inertia ixx="1" ixy="0" ixz="0" iyy="1" iyz="0" izz="1" />
       </inertial>
@@ -44,18 +44,18 @@
       </visual>
     </link>
-    <joint name="dummy_to_base_link_joint" type="fixed">
-      <origin xyz="0 0 0" rpy="0 0 0" />
-      <parent link="dummy" />
-      <child link="base_link" />
-    </joint>
-    <joint name="base_link_to_cover_joint" type="fixed">
+    <joint name="base_link_to_chassis_joint" type="fixed">
       <origin xyz="0 0 0" rpy="0 0 0" />
       <parent link="base_link" />
-      <child link="cover" />
+      <child link="chassis_link" />
     </joint>
-    <gazebo reference="base_link">
+    <joint name="chassis_to_cover_joint" type="fixed">
+      <origin xyz="0 0 0" rpy="0 0 0" />
+      <parent link="chassis_link" />
+      <child link="cover_link" />
+    </joint>
+    <gazebo reference="chassis_link">
       <material>Gazebo/White</material>
     </gazebo>
-    <gazebo reference="cover">
+    <gazebo reference="cover_link">
       <material>Gazebo/Red</material>
     </gazebo>

File: src/panther_description/urdf/gazebo_plugins.gazebo.xacro (robot description, xacro)
@@ -1,26 +1,28 @@
 <?xml version="1.0"?>
 <robot xmlns:xacro="http://www.ros.org/wiki/xacro">
-  <xacro:macro name="skid_drive" params="wheel_props common_props">
-    <gazebo>
-      <plugin name="skid_steer_drive_controller" filename="libgazebo_ros_skid_steer_drive.so">
-        <updateRate>10.0</updateRate>
-        <robotBaseFrame>base_link</robotBaseFrame>
-        <wheelSeparation>${common_props['base_link']['wheel_separation']}</wheelSeparation>
-        <wheelDiameter>${wheel_props['diameter']}</wheelDiameter>
-        <torque>${common_props['motors']['max_torque']}</torque>
-        <leftFrontJoint>front_left_wheel_joint</leftFrontJoint>
-        <rightFrontJoint>front_right_wheel_joint</rightFrontJoint>
-        <leftRearJoint>rear_left_wheel_joint</leftRearJoint>
-        <rightRearJoint>rear_right_wheel_joint</rightRearJoint>
-        <topicName>cmd_vel</topicName>
-        <commandTopic>cmd_vel</commandTopic>
-        <broadcastTF>true</broadcastTF>
-        <odometryTopic>odom</odometryTopic>
-        <odometryFrame>odom</odometryFrame>
-        <covariance_x>0.000100</covariance_x>
-        <covariance_y>0.000100</covariance_y>
-        <covariance_yaw>0.010000</covariance_yaw>
-      </plugin>
-    </gazebo>
+  <xacro:macro name="wheel_driver" params="wheel_props common_props">
+    <xacro:if value="${wheel_props['simulation']['driver'] == 'skid_steer_drive_controller'}">
+      <gazebo>
+        <plugin name="skid_steer_drive_controller" filename="libgazebo_ros_skid_steer_drive.so">
+          <updateRate>10.0</updateRate>
+          <robotBaseFrame>base_link</robotBaseFrame>
+          <wheelSeparation>${common_props['chassis']['wheel_separation']}</wheelSeparation>
+          <wheelDiameter>${wheel_props['front_wheels']['diameter']}</wheelDiameter>
+          <torque>${common_props['motors']['max_torque']}</torque>
+          <leftFrontJoint>front_left_wheel_joint</leftFrontJoint>
+          <rightFrontJoint>front_right_wheel_joint</rightFrontJoint>
+          <leftRearJoint>rear_left_wheel_joint</leftRearJoint>
+          <rightRearJoint>rear_right_wheel_joint</rightRearJoint>
+          <topicName>cmd_vel</topicName>
+          <commandTopic>cmd_vel</commandTopic>
+          <broadcastTF>true</broadcastTF>
+          <odometryTopic>odom</odometryTopic>
+          <odometryFrame>odom</odometryFrame>
+          <covariance_x>0.000100</covariance_x>
+          <covariance_y>0.000100</covariance_y>
+          <covariance_yaw>0.010000</covariance_yaw>
+        </plugin>
+      </gazebo>
+    </xacro:if>
   </xacro:macro>
 </robot>

File: src/panther_description/urdf/panther.urdf.xacro (robot description, xacro)
@@ -9,9 +9,9 @@
   <xacro:property name="wheel_props" value="${load_yaml(wheel_props_file)}" />
   <!-- INCLUDE ROBOT PARTS DEFINITIONS -->
-  <xacro:include filename="$(find panther_description)/urdf/base_link.urdf.xacro" ns="base_link" />
+  <xacro:include filename="$(find panther_description)/urdf/chassis.urdf.xacro" ns="chassis" />
   <xacro:include filename="$(find panther_description)/urdf/wheel.urdf.xacro" ns="wheel" />
   <xacro:include filename="$(find panther_description)/urdf/gazebo_plugins.gazebo.xacro" ns="gazebo" />
   <!-- BODY DECLARATION -->
-  <xacro:base_link.base_link props="${panther_common_props['base_link']}" />
+  <xacro:chassis.chassis props="${panther_common_props['chassis']}" />
   <!-- WHEEL DECLARATION -->
   <xacro:wheel.wheel wheel_props="${wheel_props['front_wheels']}" common_props="${panther_common_props}" prefix="front_left" />
@@ -20,8 +20,9 @@
   <xacro:wheel.wheel wheel_props="${wheel_props['rear_wheels']}"  common_props="${panther_common_props}" prefix="rear_right" />
   <!-- GAZEBO PLUGINS -->
-  <xacro:gazebo.skid_drive wheel_props="${wheel_props['front_wheels']}" common_props="${panther_common_props}" />
+  <xacro:gazebo.wheel_driver wheel_props="${wheel_props}" common_props="${panther_common_props}" />
   <gazebo>
     <plugin name="gazebo_ros_control" filename="libgazebo_ros_control.so">
       <robotNamespace>/</robotNamespace>
+      <legacyModeNS>true</legacyModeNS>
     </plugin>
   </gazebo>

File: src/panther_description/urdf/wheel.urdf.xacro (robot description, xacro)
@@ -6,17 +6,17 @@
     <xacro:if value="${prefix == 'front_left'}">
       <xacro:property name="x" value="0.38" />
-      <xacro:property name="y" value="${common_props['base_link']['wheel_separation']/2}" />
+      <xacro:property name="y" value="${common_props['chassis']['wheel_separation']/2}" />
     </xacro:if>
     <xacro:if value="${prefix == 'front_right'}">
       <xacro:property name="x" value="0.38" />
-      <xacro:property name="y" value="-${common_props['base_link']['wheel_separation']/2}" />
+      <xacro:property name="y" value="-${common_props['chassis']['wheel_separation']/2}" />
     </xacro:if>
     <xacro:if value="${prefix == 'rear_left'}">
       <xacro:property name="x" value="-0.38" />
-      <xacro:property name="y" value="${common_props['base_link']['wheel_separation']/2}" />
+      <xacro:property name="y" value="${common_props['chassis']['wheel_separation']/2}" />
     </xacro:if>
     <xacro:if value="${prefix == 'rear_right'}">
       <xacro:property name="x" value="-0.38" />
-      <xacro:property name="y" value="-${common_props['base_link']['wheel_separation']/2}" />
+      <xacro:property name="y" value="-${common_props['chassis']['wheel_separation']/2}" />
     </xacro:if>
     <link name="${prefix}_wheel_link">
@@ -47,8 +47,8 @@
     </link>
     <joint name="${prefix}_wheel_joint" type="continuous">
-      <parent link="base_link" />
+      <parent link="chassis_link" />
       <child link="${prefix}_wheel_link" />
       <origin xyz="${x} ${y} 0" rpy="0 0 0" />
-      <axis xyz="1 0 0" />
+      <axis xyz="0 1 0" />
       <limit effort="${common_props['motors']['max_torque']}"
              velocity="${common_props['motors']['max_velocity']}" />
@@ -56,11 +56,12 @@
                 friction="${common_props['motors']['joint_friction']}"/>
     </joint>
-    <transmission name="${prefix}_wheel_transmission">
+    <transmission name="${prefix}_wheel_transmission" type="SimpleTransmission">
       <type>transmission_interface/SimpleTransmission</type>
       <joint name="${prefix}_wheel_joint">
         <hardwareInterface>hardware_interface/EffortJointInterface</hardwareInterface>
       </joint>
-      <actuator name="${prefix}_actuator">
+      <actuator name="${prefix}_wheel_actuator">
         <mechanicalReduction>1</mechanicalReduction>
+        <hardwareInterface>hardware_interface/EffortJointInterface</hardwareInterface>
       </actuator>
     </transmission>

Commit message: Add rplidar s1 component

File: src/panther_description/urdf/chassis.urdf.xacro (robot description, xacro)
@@ -11,10 +11,10 @@
         </geometry>
         <origin xyz="0 0 0" rpy=" ${pi/2} 0 ${pi/2}"/>
-        <material name="base_color"> <color rgba="${props['visual']['base']['color_rgb']} 1.0"/> </material>
+        <material name="${props['visual']['base']['color']}"/>
       </visual>
       <collision>
         <geometry>
             <xacro:property name="mesh" value="${props['collision']['mesh']}" />
-          <mesh filename="package://panther_description/meshes/${mesh}" scale="0.001 0.001 0.001" />
+            <mesh filename="package://panther_description/meshes/${mesh}" scale="0.001 0.001 0.001" />
         </geometry>
         <origin xyz="0 0 0" rpy=" ${pi/2} 0 ${pi/2}"/>
@@ -41,5 +41,5 @@
         </geometry>
         <origin xyz="0 0 0" rpy=" ${pi/2} 0 ${pi/2}"/>
-        <material name="cover_color"> <color rgba="${props['visual']['cover']['color_rgb']} 1.0"/> </material>
+        <material name="${props['visual']['cover']['color']}"/>
       </visual>
     </link>
@@ -55,8 +55,8 @@
     </joint>
     <gazebo reference="chassis_link">
-      <material>Gazebo/White</material>
+      <material>Gazebo/${props['visual']['base']['color']}</material>
     </gazebo>
     <gazebo reference="cover_link">
-      <material>Gazebo/Red</material>
+      <material>Gazebo/${props['visual']['cover']['color']}</material>
     </gazebo>
   </xacro:macro>

File: src/panther_description/urdf/gazebo_plugins.gazebo.xacro (robot description, xacro)
@@ -1,4 +1,5 @@
 <?xml version="1.0"?>
 <robot xmlns:xacro="http://www.ros.org/wiki/xacro">
+  <xacro:include filename="$(find panther_description)/urdf/components/rplidar_s1.gazebo.xacro" />
   <xacro:macro name="wheel_driver" params="wheel_props common_props">
     <xacro:if value="${wheel_props['simulation']['driver'] == 'skid_steer_drive_controller'}">

File: src/panther_description/urdf/panther.urdf.xacro (robot description, xacro)
@@ -3,4 +3,5 @@
   <xacro:arg name="panther_common_props_path" default="$(find panther_description)/config/panther_common.yaml" />
   <xacro:arg name="wheel_props_path" default="$(find panther_description)/config/classic_wheels_props.yaml" />
+  <xacro:arg name="use_gpu" default="false" />
   <!-- IMPORT YAML CONFIGS -->
   <xacro:property name="panther_common_props_file" value="$(arg panther_common_props_path)"  />
@@ -9,4 +10,5 @@
   <xacro:property name="wheel_props" value="${load_yaml(wheel_props_file)}" />
   <!-- INCLUDE ROBOT PARTS DEFINITIONS -->
+  <xacro:include filename="$(find panther_description)/urdf/materials.urdf.xacro" />
   <xacro:include filename="$(find panther_description)/urdf/chassis.urdf.xacro" ns="chassis" />
   <xacro:include filename="$(find panther_description)/urdf/wheel.urdf.xacro" ns="wheel" />
@@ -21,4 +23,5 @@
   <!-- GAZEBO PLUGINS -->
   <xacro:gazebo.wheel_driver wheel_props="${wheel_props}" common_props="${panther_common_props}" />
+  <xacro:gazebo.rplidar_s1 xyz="0.2 0 0.14" rpy="0 0 0" use_gpu="$(arg use_gpu)" />
   <gazebo>
     <plugin name="gazebo_ros_control" filename="libgazebo_ros_control.so">

File: src/panther_description/urdf/wheel.urdf.xacro (robot description, xacro)
@@ -27,5 +27,5 @@
         </geometry>
         <origin xyz="0 0 0" rpy="${rpy}"/>
-        <material name="wheel_color"> <color rgba="${wheel_props['color_rgb']} 1.0"/> </material>
+        <material name="${wheel_props['color']}"/>
       </visual>
       <collision>
@@ -72,5 +72,5 @@
       <kd value="${wheel_props['contact_damping']}" />
       <fdir1 value="1 0 0"/>
-      <material>Gazebo/Grey</material>
+      <material>Gazebo/${wheel_props['color']}</material>
     </gazebo>
     <gazebo reference="${prefix}_wheel_joint">
