Commit message: Accurate meshes

File: src/panther_description/urdf/body.urdf.xacro (robot description, xacro)
@@ -1,12 +1,12 @@
 <?xml version="1.0" encoding="utf-8"?>
 <robot xmlns:xacro="http://www.ros.org/wiki/xacro">
-  <!-- chassis defining macro -->
-  <xacro:macro name="chassis" params="props">
+  <!-- body defining macro -->
+  <xacro:macro name="body" params="props">
     <link name="base_link"></link>
-    <link name="chassis_link">
+    <link name="body_link">
       <visual>
         <geometry>
             <xacro:property name="mesh" value="${props['visual']['base']['mesh']}" />
-            <mesh filename="package://panther_description/meshes/${mesh}" scale="0.001 0.001 0.001" />
+            <mesh filename="package://panther_description/meshes/${mesh}" scale="1 1 1" />
         </geometry>
         <origin xyz="0 0 0" rpy=" ${pi/2} 0 ${pi/2}"/>
@@ -16,5 +16,5 @@
         <geometry>
             <xacro:property name="mesh" value="${props['collision']['mesh']}" />
-            <mesh filename="package://panther_description/meshes/${mesh}" scale="0.001 0.001 0.001" />
+            <mesh filename="package://panther_description/meshes/${mesh}" scale="1 1 1" />
         </geometry>
         <origin xyz="0 0 0" rpy=" ${pi/2} 0 ${pi/2}"/>
@@ -38,5 +38,5 @@
         <geometry>
           <xacro:property name="mesh" value="${props['visual']['cover']['mesh']}" />
-          <mesh filename="package://panther_description/meshes/${mesh}" scale="0.001 0.001 0.001" />
+          <mesh filename="package://panther_description/meshes/${mesh}" scale="1 1 1" />
         </geometry>
         <origin xyz="0 0 0" rpy=" ${pi/2} 0 ${pi/2}"/>
@@ -44,15 +44,34 @@
       </visual>
     </link>
-    <joint name="base_link_to_chassis_joint" type="fixed">
+    <link name="rails_link">
+      <inertial>
+        <mass value="0.0000001" />
+        <inertia ixx="1" ixy="0" ixz="0" iyy="1" iyz="0" izz="1" />
+      </inertial>
+      <visual>
+        <geometry>
+          <xacro:property name="mesh" value="${props['visual']['rails']['mesh']}" />
+          <mesh filename="package://panther_description/meshes/${mesh}" scale="1 1 1" />
+        </geometry>
+        <origin xyz="0 0 0" rpy=" ${pi/2} 0 ${pi/2}"/>
+        <material name="${props['visual']['rails']['color']}"/>
+      </visual>
+    </link>
+    <joint name="base_link_to_body_joint" type="fixed">
       <origin xyz="0 0 0" rpy="0 0 0" />
       <parent link="base_link" />
-      <child link="chassis_link" />
+      <child link="body_link" />
     </joint>
-    <joint name="chassis_to_cover_joint" type="fixed">
+    <joint name="body_to_cover_joint" type="fixed">
       <origin xyz="0 0 0" rpy="0 0 0" />
-      <parent link="chassis_link" />
+      <parent link="body_link" />
       <child link="cover_link" />
     </joint>
-    <gazebo reference="chassis_link">
+    <joint name="body_to_rails_joint" type="fixed">
+      <origin xyz="0 0 0" rpy="0 0 0" />
+      <parent link="body_link" />
+      <child link="rails_link" />
+    </joint>
+    <gazebo reference="body_link">
       <material>Gazebo/${props['visual']['base']['color']}</material>
     </gazebo>
@@ -60,4 +79,7 @@
       <material>Gazebo/${props['visual']['cover']['color']}</material>
     </gazebo>
+    <gazebo reference="rails_link">
+      <material>Gazebo/${props['visual']['rails']['color']}</material>
+    </gazebo>
   </xacro:macro>
 </robot>

File: src/panther_description/urdf/components/orbebec_astra.gazebo.xacro (robot description, xacro)
@@ -7,12 +7,12 @@
             <mesh filename="package://panther_description/meshes/components/orbebec_astra.dae" scale="0.001 0.001 0.001" />
         </geometry>
-        <origin xyz="-0.01 0 -0.03" rpy="${pi/2} 0 ${pi/2}"/>
+        <origin xyz="-0.01 0 0.025" rpy="${pi/2} 0 ${pi/2}"/>
         <material name="DarkGrey"/>
       </visual>
       <collision>
         <geometry>
-          <box size="0.165 0.03 0.04" />
+          <box size="0.165 0.04 0.05" />
         </geometry>
-        <origin xyz="0 0 0.02" rpy="0 0 0"/>
+        <origin xyz="-0.01 0 0.025" rpy="0 0 ${pi/2}"/>
       </collision>
       <inertial>
@@ -21,8 +21,14 @@
       </inertial>
     </link>
+    <link name="${prefix}_orbebec_astra_depth_link"></link>
     <joint name="base_link_to_${prefix}_orbebec_astra_link_joint" type="fixed">
       <origin xyz="${xyz}" rpy="${rpy}" />
       <parent link="base_link" />
       <child link="${prefix}_orbebec_astra_link" />
+    </joint>
+    <joint name="${prefix}_orbebec_astra_depth_link_joint" type="fixed">
+      <origin xyz="0.01 0 0.035" rpy="${-pi/2} 0 ${-pi/2}" />
+      <parent link="${prefix}_orbebec_astra_link" />
+      <child link="${prefix}_orbebec_astra_depth_link" />
     </joint>
     <gazebo reference="${prefix}_orbebec_astra_link">
@@ -51,5 +57,5 @@
           <updateRate>10.0</updateRate>
           <cameraName>camera</cameraName>
-          <frameName>camera_depth_frame</frameName>
+          <frameName>${prefix}_orbebec_astra_depth_link</frameName>
           <imageTopicName>rgb/image_raw</imageTopicName>
           <depthImageTopicName>depth/image_raw</depthImageTopicName>

File: src/panther_description/urdf/components/ouster_os1_32.gazebo.xacro (robot description, xacro)
@@ -1,5 +1,5 @@
 <?xml version="1.0"?>
 <robot xmlns:xacro="http://www.ros.org/wiki/xacro">
-  <xacro:macro name="ouster_os1_16" params="xyz rpy use_gpu:=false prefix:=front topic:=laser/scan">
+  <xacro:macro name="ouster_os1_32" params="xyz rpy use_gpu:=false prefix:=front topic:=laser/scan">
     <xacro:if value="${use_gpu}">
       <xacro:property name="ray_type" value="gpu_ray" />
@@ -10,8 +10,8 @@
       <xacro:property name="plugin_file_name" value="libgazebo_ros_laser.so" />
     </xacro:unless>
-    <link name="${prefix}_ouster_os1_16_link">
+    <link name="${prefix}_ouster_os1_32_link">
       <visual>
         <geometry>
-          <!-- <mesh filename="package://panther_description/meshes/components/ouster_os1_16.stl" scale="0.0001 0.0001 0.0001" /> -->
+          <!-- <mesh filename="package://panther_description/meshes/components/ouster_os1_32.stl" scale="0.0001 0.0001 0.0001" /> -->
           <cylinder radius="${0.0555/2}" length="0.051" />
         </geometry>
@@ -30,20 +30,20 @@
       </inertial>
     </link>
-    <link name="${prefix}_ouster_os1_16_laser_link"></link>
-    <joint name="base_link_to_${prefix}_ouster_os1_16_link_joint" type="fixed">
+    <link name="${prefix}_ouster_os1_32_laser_link"></link>
+    <joint name="base_link_to_${prefix}_ouster_os1_32_link_joint" type="fixed">
       <origin xyz="${xyz}" rpy="${rpy}" />
       <parent link="base_link" />
-      <child link="${prefix}_ouster_os1_16_link" />
+      <child link="${prefix}_ouster_os1_32_link" />
     </joint>
-    <joint name="${prefix}_ouster_os1_16_laser_link_joint" type="fixed">
+    <joint name="${prefix}_ouster_os1_32_laser_link_joint" type="fixed">
       <origin xyz="0 0 0.0378" rpy="0 0 0" />
-      <parent link="${prefix}_ouster_os1_16_link" />
-      <child link="${prefix}_ouster_os1_16_laser_link" />
+      <parent link="${prefix}_ouster_os1_32_link" />
+      <child link="${prefix}_ouster_os1_32_laser_link" />
     </joint>
-    <gazebo reference="${prefix}_ouster_os1_16_link">
+    <gazebo reference="${prefix}_ouster_os1_32_link">
       <material>Gazebo/DarkGrey</material>
     </gazebo>
-    <gazebo reference="${prefix}_ouster_os1_16_laser_link">
-      <sensor type="${ray_type}" name="${prefix}_ouster_os1_16_sensor">
+    <gazebo reference="${prefix}_ouster_os1_32_laser_link">
+      <sensor type="${ray_type}" name="${prefix}_ouster_os1_32_sensor">
         <pose>0 0 0.0 0 0 0</pose>
         <visualize>false</visualize>
@@ -58,5 +58,5 @@
             </horizontal>
             <vertical>
-              <samples>128</samples>
+              <samples>32</samples>
               <resolution>1</resolution>
               <min_angle>-${25.5/180*pi}</min_angle>
@@ -65,5 +65,5 @@
           </scan>
           <range>
-            <min>0.2</min>
+            <min>0.05</min>
             <max>120.0</max>
             <resolution>0.007</resolution>
@@ -71,5 +71,5 @@
           <noise>
             <type>gaussian</type>
-            <mean>0.05</mean>
+            <mean>0.0</mean>
             <stddev>0.007</stddev>
           </noise>
@@ -77,5 +77,5 @@
         <plugin name="gazebo_ros_head_rplidar_controller" filename="${plugin_file_name}">
           <topicName>${topic}</topicName>
-          <frameName>${prefix}_ouster_os1_16_laser_link</frameName>
+          <frameName>${prefix}_ouster_os1_32_laser_link</frameName>
         </plugin>
       </sensor>

File: src/panther_description/urdf/components/rplidar_s1.gazebo.xacro (robot description, xacro)
@@ -60,10 +60,10 @@
             <min>0.1</min>
             <max>40.0</max>
-            <resolution>0.03</resolution>
+            <resolution>0.015</resolution>
           </range>
           <noise>
             <type>gaussian</type>
             <mean>0</mean>
-            <stddev>0.03</stddev>
+            <stddev>0.00125</stddev>
           </noise>
         </ray>

File: src/panther_description/urdf/components/velodyne_puck.gazebo.xacro (robot description, xacro)
@@ -66,5 +66,5 @@
             <min>0.2</min>
             <max>100.0</max>
-            <resolution>0.03</resolution>
+            <resolution>0.015</resolution>
           </range>
           <noise>

File: src/panther_description/urdf/gazebo_plugins.gazebo.xacro (robot description, xacro)
@@ -5,6 +5,6 @@
   <xacro:include filename="$(find panther_description)/urdf/components/rplidar_a3.gazebo.xacro" />
   <xacro:include filename="$(find panther_description)/urdf/components/velodyne_puck.gazebo.xacro" />
+  <xacro:include filename="$(find panther_description)/urdf/components/ouster_os1_32.gazebo.xacro" />
   <xacro:include filename="$(find panther_description)/urdf/components/orbebec_astra.gazebo.xacro" />
-  <xacro:include filename="$(find panther_description)/urdf/components/ouster_os1_16.gazebo.xacro" />
   <xacro:macro name="wheel_driver" params="wheel_props common_props">
     <xacro:if value="${wheel_props['simulation']['driver'] == 'libgazebo_ros_skid_steer_drive'}">
@@ -13,6 +13,6 @@
           <updateRate>10.0</updateRate>
           <robotBaseFrame>base_link</robotBaseFrame>
-          <wheelSeparation>${common_props['chassis']['wheel_separation']}</wheelSeparation>
-          <wheelDiameter>${wheel_props['front_wheels']['diameter']}</wheelDiameter>
+          <wheelSeparation>${common_props['body']['wheel_separation']}</wheelSeparation>
+          <wheelDiameter>${wheel_props['wheels']['diameter']}</wheelDiameter>
           <torque>${common_props['motors']['max_torque']}</torque>
           <leftFrontJoint>front_left_wheel_joint</leftFrontJoint>

File: src/panther_description/urdf/panther.urdf.xacro (robot description, xacro)
@@ -3,5 +3,5 @@
   <xacro:arg name="panther_common_props_path" default="$(find panther_description)/config/panther_common.yaml" />
   <xacro:arg name="wheel_props_path" default="$(find panther_description)/config/classic_wheels_props.yaml" />
-  <xacro:arg name="use_gpu" default="true" />
+  <xacro:arg name="use_gpu" default="false" />
   <!-- IMPORT YAML CONFIGS -->
   <xacro:property name="panther_common_props_file" value="$(arg panther_common_props_path)"  />
@@ -11,17 +11,17 @@
   <!-- INCLUDE ROBOT PARTS DEFINITIONS -->
   <xacro:include filename="$(find panther_description)/urdf/materials.urdf.xacro" />
-  <xacro:include filename="$(find panther_description)/urdf/chassis.urdf.xacro" ns="chassis" />
+  <xacro:include filename="$(find panther_description)/urdf/body.urdf.xacro" ns="body" />
   <xacro:include filename="$(find panther_description)/urdf/wheel.urdf.xacro" ns="wheel" />
   <xacro:include filename="$(find panther_description)/urdf/gazebo_plugins.gazebo.xacro" ns="gazebo" />
   <!-- BODY DECLARATION -->
-  <xacro:chassis.chassis props="${panther_common_props['chassis']}" />
+  <xacro:body.body props="${panther_common_props['body']}" />
   <!-- WHEEL DECLARATION -->
-  <xacro:wheel.wheel wheel_props="${wheel_props['front_wheels']}" common_props="${panther_common_props}" prefix="front_left" />
-  <xacro:wheel.wheel wheel_props="${wheel_props['front_wheels']}" common_props="${panther_common_props}" prefix="front_right" />
-  <xacro:wheel.wheel wheel_props="${wheel_props['rear_wheels']}"  common_props="${panther_common_props}" prefix="rear_left" />
-  <xacro:wheel.wheel wheel_props="${wheel_props['rear_wheels']}"  common_props="${panther_common_props}" prefix="rear_right" />
+  <xacro:wheel.wheel wheel_props="${wheel_props['wheels']}" common_props="${panther_common_props}" prefix="front_left" />
+  <xacro:wheel.wheel wheel_props="${wheel_props['wheels']}" common_props="${panther_common_props}" prefix="front_right" />
+  <xacro:wheel.wheel wheel_props="${wheel_props['wheels']}"  common_props="${panther_common_props}" prefix="rear_left" />
+  <xacro:wheel.wheel wheel_props="${wheel_props['wheels']}"  common_props="${panther_common_props}" prefix="rear_right" />
   <!-- GAZEBO PLUGINS -->
   <xacro:gazebo.wheel_driver wheel_props="${wheel_props}" common_props="${panther_common_props}" />
-  <xacro:gazebo.rplidar_s1 xyz="0.2 0 0.2" rpy="0 0 0" use_gpu="true" />
+  <xacro:gazebo.rplidar_s1 xyz="0.185 0 0.17" rpy="0 0 0" use_gpu="$(arg use_gpu)" />
   <gazebo>
     <plugin name="gazebo_ros_control" filename="libgazebo_ros_control.so">

File: src/panther_description/urdf/wheel.urdf.xacro (robot description, xacro)
@@ -5,24 +5,27 @@
     <xacro:property name="rpy" value="0 0 ${pi/2}" />
     <xacro:if value="${prefix == 'front_left'}">
-      <xacro:property name="x" value="0.38" />
-      <xacro:property name="y" value="${common_props['chassis']['wheel_separation']/2}" />
+      <xacro:property name="x" value="0.22" />
+      <xacro:property name="y" value="${common_props['body']['wheel_separation']/2}" />
+      <xacro:property name="mesh" value="${wheel_props['visual_mesh_left']}" />
     </xacro:if>
     <xacro:if value="${prefix == 'front_right'}">
-      <xacro:property name="x" value="0.38" />
-      <xacro:property name="y" value="-${common_props['chassis']['wheel_separation']/2}" />
+      <xacro:property name="x" value="0.22" />
+      <xacro:property name="y" value="-${common_props['body']['wheel_separation']/2}" />
+      <xacro:property name="mesh" value="${wheel_props['visual_mesh_right']}" />
     </xacro:if>
     <xacro:if value="${prefix == 'rear_left'}">
-      <xacro:property name="x" value="-0.38" />
-      <xacro:property name="y" value="${common_props['chassis']['wheel_separation']/2}" />
+      <xacro:property name="x" value="-0.22" />
+      <xacro:property name="y" value="${common_props['body']['wheel_separation']/2}" />
+      <xacro:property name="mesh" value="${wheel_props['visual_mesh_left']}" />
     </xacro:if>
     <xacro:if value="${prefix == 'rear_right'}">
-      <xacro:property name="x" value="-0.38" />
-      <xacro:property name="y" value="-${common_props['chassis']['wheel_separation']/2}" />
+      <xacro:property name="x" value="-0.22" />
+      <xacro:property name="y" value="-${common_props['body']['wheel_separation']/2}" />
+      <xacro:property name="mesh" value="${wheel_props['visual_mesh_right']}" />
     </xacro:if>
     <link name="${prefix}_wheel_link">
        <visual>
         <geometry>
-            <xacro:property name="mesh" value="${wheel_props['visual_mesh']}" />
-            <mesh filename="package://panther_description/meshes/${mesh}" scale="0.001 0.001 0.001" />
+            <mesh filename="package://panther_description/meshes/${mesh}" scale="1 1 1" />
         </geometry>
         <origin xyz="0 0 0" rpy="${rpy}"/>
@@ -32,5 +35,5 @@
         <geometry>
             <xacro:property name="mesh" value="${wheel_props['collision_mesh']}" />
-            <mesh filename="package://panther_description/meshes/${mesh}" scale="0.001 0.001 0.001" />
+            <mesh filename="package://panther_description/meshes/${mesh}" scale="1 1 1" />
         </geometry>
         <origin xyz="0 0 0" rpy="${rpy}" />
@@ -47,5 +50,5 @@
     </link>
     <joint name="${prefix}_wheel_joint" type="continuous">
-      <parent link="chassis_link" />
+      <parent link="body_link" />
       <child link="${prefix}_wheel_link" />
       <origin xyz="${x} ${y} 0" rpy="0 0 0" />
