Commit message: All wheel type  | IMU and GPS from hector plugins

File: src/panther_description/urdf/body.urdf.xacro (robot description, xacro)
@@ -58,4 +58,16 @@
       </visual>
     </link>
+    <link name="imu_link">
+      <inertial>
+        <mass value="0.0000001" />
+        <inertia ixx="1" ixy="0" ixz="0" iyy="1" iyz="0" izz="1" />
+      </inertial>
+    </link>
+    <link name="gps_link">
+      <inertial>
+        <mass value="0.0000001" />
+        <inertia ixx="1" ixy="0" ixz="0" iyy="1" iyz="0" izz="1" />
+      </inertial>
+    </link>
     <joint name="base_link_to_body_joint" type="fixed">
       <origin xyz="0 0 0" rpy="0 0 0" />
@@ -73,4 +85,14 @@
       <child link="rails_link" />
     </joint>
+    <joint name="base_link_to_imu_link_joint" type="fixed">
+      <origin xyz="0.169 0.025 0.092" rpy="0 0 0" />
+      <parent link="base_link" />
+      <child link="imu_link" />
+    </joint>
+    <joint name="base_link_to_gps_link_joint" type="fixed">
+      <origin xyz="0.169 0.025 0.092" rpy="0 0 0" />
+      <parent link="base_link" />
+      <child link="gps_link" />
+    </joint>
     <gazebo reference="body_link">
       <material>Gazebo/${props['visual']['base']['color']}</material>

File: src/panther_description/urdf/gazebo_plugins.gazebo.xacro (robot description, xacro)
@@ -13,5 +13,5 @@
           <updateRate>10.0</updateRate>
           <robotBaseFrame>base_link</robotBaseFrame>
-          <wheelSeparation>${common_props['body']['wheel_separation']}</wheelSeparation>
+          <wheelSeparation>${wheel_props['wheels']['wheel_separation']}</wheelSeparation>
           <wheelDiameter>${wheel_props['wheels']['diameter']}</wheelDiameter>
           <torque>${common_props['motors']['max_torque']}</torque>
@@ -43,34 +43,37 @@
       </gazebo>
     </xacro:if>
-    <link name="imu">
-      <inertial>
-        <mass value="0.0000001" />
-        <inertia ixx="1" ixy="0" ixz="0" iyy="1" iyz="0" izz="1" />
-      </inertial>
-    </link>
-    <joint name="base_link_to_imu_link_joint" type="fixed">
-      <origin xyz="0.169 0.025 0.092" rpy="0 0 0" />
-      <parent link="base_link" />
-      <child link="imu" />
-    </joint>
-    <gazebo reference="imu">
-      <gravity>true</gravity>
-      <sensor name="imu_sensor" type="imu">
-        <always_on>true</always_on>
-        <update_rate>100</update_rate>
-        <visualize>false</visualize>
-        <topic>imu/data</topic>
-        <plugin filename="libgazebo_ros_imu_sensor.so" name="imu_plugin">
-          <topicName>imu/data</topicName>
-          <bodyName>imu</bodyName>
-          <updateRateHZ>125.0</updateRateHZ>
-          <gaussianNoise>${0.095*(pi/180.0)}</gaussianNoise>
-          <xyzOffset>0 0 0</xyzOffset>
-          <rpyOffset>0 0 0</rpyOffset>
-          <frameName>imu</frameName>
-          <initialOrientationAsReference>false</initialOrientationAsReference>
-        </plugin>
-        <pose>0 0 0 0 0 0</pose>
-      </sensor>
+    <!-- based on PhidgetSpatial datasheet -->
+    <xacro:property name="imu_acc_noise"  value="${280.0*1e-6*9.81}" />
+    <xacro:property name="imu_acc_drift"  value="${40.6*1e-6*9.81}" />
+    <xacro:property name="imu_gyro_noise" value="${0.095*(pi/180.0)}" />
+    <xacro:property name="imu_gyro_drift" value="${0.0042*(pi/180.0)}" />
+    <gazebo>
+      <plugin name="imu_controller" filename="libhector_gazebo_ros_imu.so">
+        <robotNamespace>/</robotNamespace>
+        <updateRate>100.0</updateRate>
+        <bodyName>imu_link</bodyName>
+        <topicName>imu</topicName>
+        <accelDrift>${imu_acc_drift} ${imu_acc_drift} ${imu_acc_drift}</accelDrift>
+        <accelGaussianNoise>${imu_acc_noise} ${imu_acc_noise} ${imu_acc_noise}</accelGaussianNoise>
+        <rateDrift>${imu_gyro_drift} ${imu_gyro_drift} ${imu_gyro_drift}</rateDrift>
+        <rateGaussianNoise>${imu_gyro_noise} ${imu_gyro_noise} ${imu_gyro_noise}</rateGaussianNoise>
+      </plugin>
+    </gazebo>
+    <!-- based on Teltonika RUTX11 datasheet and measuremets-->
+    <gazebo>
+      <plugin name="gps_controller" filename="libhector_gazebo_ros_gps.so">
+        <updateRate>40</updateRate>
+        <robotNamespace>/</robotNamespace>
+        <bodyName>gps_link</bodyName>
+        <frameId>gps_link</frameId>
+        <topicName>/global_position/fix</topicName>
+        <velocityTopicName>/global_position/vel</velocityTopicName>
+        <referenceLatitude>53.1978</referenceLatitude>
+        <referenceLongitude>18.3735</referenceLongitude>
+        <referenceHeading>0</referenceHeading>
+        <referenceAltitude>0</referenceAltitude>
+        <drift>0.0001 0.0001 0.0001</drift>
+        <gaussianNoise>3.0 3.0 3.0</gaussianNoise>
+      </plugin>
     </gazebo>
   </xacro:macro>

File: src/panther_description/urdf/panther.urdf.xacro (robot description, xacro)
@@ -19,6 +19,6 @@
   <xacro:wheel.wheel wheel_props="${wheel_props['wheels']}" common_props="${panther_common_props}" prefix="front_left" />
   <xacro:wheel.wheel wheel_props="${wheel_props['wheels']}" common_props="${panther_common_props}" prefix="front_right" />
-  <xacro:wheel.wheel wheel_props="${wheel_props['wheels']}"  common_props="${panther_common_props}" prefix="rear_left" />
-  <xacro:wheel.wheel wheel_props="${wheel_props['wheels']}"  common_props="${panther_common_props}" prefix="rear_right" />
+  <xacro:wheel.wheel wheel_props="${wheel_props['wheels']}" common_props="${panther_common_props}" prefix="rear_left" />
+  <xacro:wheel.wheel wheel_props="${wheel_props['wheels']}" common_props="${panther_common_props}" prefix="rear_right" />
   <!-- GAZEBO PLUGINS -->
   <xacro:gazebo.wheel_driver wheel_props="${wheel_props}" common_props="${panther_common_props}" />

File: src/panther_description/urdf/wheel.urdf.xacro (robot description, xacro)
@@ -4,28 +4,29 @@
   <xacro:macro name="wheel" params="wheel_props common_props prefix">
     <xacro:property name="rpy" value="0 0 ${pi/2}" />
+    <xacro:property name="mesh_folder" value="${wheel_props['mesh_folder']}" />
     <xacro:if value="${prefix == 'front_left'}">
       <xacro:property name="x" value="0.22" />
-      <xacro:property name="y" value="${common_props['body']['wheel_separation']/2}" />
-      <xacro:property name="mesh" value="${wheel_props['visual_mesh_left']}" />
+      <xacro:property name="y" value="${wheel_props['wheel_separation']/2}" />
+      <xacro:property name="mesh" value="package://panther_description/meshes/${mesh_folder}/wheel_a.stl" />
     </xacro:if>
     <xacro:if value="${prefix == 'front_right'}">
       <xacro:property name="x" value="0.22" />
-      <xacro:property name="y" value="-${common_props['body']['wheel_separation']/2}" />
-      <xacro:property name="mesh" value="${wheel_props['visual_mesh_right']}" />
+      <xacro:property name="y" value="-${wheel_props['wheel_separation']/2}" />
+      <xacro:property name="mesh" value="package://panther_description/meshes/${mesh_folder}/wheel_b.stl" />
     </xacro:if>
     <xacro:if value="${prefix == 'rear_left'}">
       <xacro:property name="x" value="-0.22" />
-      <xacro:property name="y" value="${common_props['body']['wheel_separation']/2}" />
-      <xacro:property name="mesh" value="${wheel_props['visual_mesh_left']}" />
+      <xacro:property name="y" value="${wheel_props['wheel_separation']/2}" />
+      <xacro:property name="mesh" value="package://panther_description/meshes/${mesh_folder}/wheel_a.stl" />
     </xacro:if>
     <xacro:if value="${prefix == 'rear_right'}">
       <xacro:property name="x" value="-0.22" />
-      <xacro:property name="y" value="-${common_props['body']['wheel_separation']/2}" />
-      <xacro:property name="mesh" value="${wheel_props['visual_mesh_right']}" />
+      <xacro:property name="y" value="-${wheel_props['wheel_separation']/2}" />
+      <xacro:property name="mesh" value="package://panther_description/meshes/${mesh_folder}/wheel_b.stl" />
     </xacro:if>
     <link name="${prefix}_wheel_link">
        <visual>
         <geometry>
-            <mesh filename="package://panther_description/meshes/${mesh}" scale="1 1 1" />
+            <mesh filename="${mesh}" scale="1 1 1" />
         </geometry>
         <origin xyz="0 0 0" rpy="${rpy}"/>
@@ -34,6 +35,5 @@
       <collision>
         <geometry>
-            <xacro:property name="mesh" value="${wheel_props['collision_mesh']}" />
-            <mesh filename="package://panther_description/meshes/${mesh}" scale="1 1 1" />
+            <mesh filename="package://panther_description/meshes/${mesh_folder}/collision.stl" scale="1 1 1" />
         </geometry>
         <origin xyz="0 0 0" rpy="${rpy}" />
