Commit message: Lidar components definitions

File: src/panther_description/urdf/components/ouster_os1_16.gazebo.xacro (robot description, xacro)
@@ -1,5 +1,5 @@
 <?xml version="1.0"?>
 <robot xmlns:xacro="http://www.ros.org/wiki/xacro">
-  <xacro:macro name="rplidar_s1" params="xyz rpy use_gpu:=false prefix:=front topic:=laser/scan">
+  <xacro:macro name="ouster_os1_16" params="xyz rpy use_gpu:=false prefix:=front topic:=laser/scan">
     <xacro:if value="${use_gpu}">
       <xacro:property name="ray_type" value="gpu_ray" />
@@ -10,8 +10,9 @@
       <xacro:property name="plugin_file_name" value="libgazebo_ros_laser.so" />
     </xacro:unless>
-    <link name="${prefix}_rplidar_s1_link">
+    <link name="${prefix}_ouster_os1_16_link">
       <visual>
         <geometry>
-          <mesh filename="package://panther_description/meshes/components/rplidar_s1.stl" scale="0.0001 0.0001 0.0001" />
+          <!-- <mesh filename="package://panther_description/meshes/components/ouster_os1_16.stl" scale="0.0001 0.0001 0.0001" /> -->
+          <cylinder radius="${0.0555/2}" length="0.051" />
         </geometry>
         <origin xyz="0 0 ${0.051/2}" rpy="0 0 -${pi/2}"/>
@@ -25,25 +26,25 @@
       </collision>
       <inertial>
-        <mass value="0.105" />
-        <inertia ixx="1" ixy="0" ixz="0" iyy="1" iyz="0" izz="1" />
+          <mass value="0.447" />
+          <inertia ixx="1" ixy="0" ixz="0" iyy="1" iyz="0" izz="1" />
       </inertial>
     </link>
-    <link name="${prefix}_rplidar_s1_laser_link"></link>
-    <joint name="base_link_to_${prefix}_rplidar_s1_link_joint" type="fixed">
+    <link name="${prefix}_ouster_os1_16_laser_link"></link>
+    <joint name="base_link_to_${prefix}_ouster_os1_16_link_joint" type="fixed">
       <origin xyz="${xyz}" rpy="${rpy}" />
       <parent link="base_link" />
-      <child link="${prefix}_rplidar_s1_link" />
+      <child link="${prefix}_ouster_os1_16_link" />
     </joint>
-    <joint name="${prefix}_rplidar_s1_laser_link_joint" type="fixed">
-      <origin xyz="0 0 0.04" rpy="0 0 0" />
-      <parent link="${prefix}_rplidar_s1_link" />
-      <child link="${prefix}_rplidar_s1_laser_link" />
+    <joint name="${prefix}_ouster_os1_16_laser_link_joint" type="fixed">
+      <origin xyz="0 0 0.0378" rpy="0 0 0" />
+      <parent link="${prefix}_ouster_os1_16_link" />
+      <child link="${prefix}_ouster_os1_16_laser_link" />
     </joint>
-    <gazebo reference="${prefix}_rplidar_s1_link">
+    <gazebo reference="${prefix}_ouster_os1_16_link">
       <material>Gazebo/DarkGrey</material>
     </gazebo>
-    <gazebo reference="${prefix}_rplidar_s1_laser_link">
-      <sensor type="${ray_type}" name="${prefix}_rplidar_s1_sensor">
-        <pose>0 0 0.04 0 0 0</pose>
+    <gazebo reference="${prefix}_ouster_os1_16_laser_link">
+      <sensor type="${ray_type}" name="${prefix}_ouster_os1_16_sensor">
+        <pose>0 0 0.0 0 0 0</pose>
         <visualize>false</visualize>
         <update_rate>10</update_rate>
@@ -51,24 +52,30 @@
           <scan>
             <horizontal>
-              <samples>9200</samples>
+              <samples>1024</samples>
               <resolution>1</resolution>
               <min_angle>-${pi}</min_angle>
               <max_angle>${pi}</max_angle>
             </horizontal>
+            <vertical>
+              <samples>128</samples>
+              <resolution>1</resolution>
+              <min_angle>-${25.5/180*pi}</min_angle>
+              <max_angle>${25.5/180*pi}</max_angle>
+            </vertical>
           </scan>
           <range>
-            <min>0.1</min>
-            <max>40.0</max>
-            <resolution>0.03</resolution>
+            <min>0.2</min>
+            <max>120.0</max>
+            <resolution>0.007</resolution>
           </range>
           <noise>
             <type>gaussian</type>
-            <mean>0</mean>
-            <stddev>0.03</stddev>
+            <mean>0.05</mean>
+            <stddev>0.007</stddev>
           </noise>
         </ray>
         <plugin name="gazebo_ros_head_rplidar_controller" filename="${plugin_file_name}">
           <topicName>${topic}</topicName>
-          <frameName>${prefix}_rplidar_s1_laser_link</frameName>
+          <frameName>${prefix}_ouster_os1_16_laser_link</frameName>
         </plugin>
       </sensor>

File: src/panther_description/urdf/components/rplidar_a2.gazebo.xacro (robot description, xacro)
@@ -1,5 +1,5 @@
 <?xml version="1.0"?>
 <robot xmlns:xacro="http://www.ros.org/wiki/xacro">
-  <xacro:macro name="rplidar_s1" params="xyz rpy use_gpu:=false prefix:=front topic:=laser/scan">
+  <xacro:macro name="rplidar_a2" params="xyz rpy use_gpu:=false prefix:=front topic:=laser/scan">
     <xacro:if value="${use_gpu}">
       <xacro:property name="ray_type" value="gpu_ray" />
@@ -10,40 +10,40 @@
       <xacro:property name="plugin_file_name" value="libgazebo_ros_laser.so" />
     </xacro:unless>
-    <link name="${prefix}_rplidar_s1_link">
+    <link name="${prefix}_rplidar_a2_link">
       <visual>
         <geometry>
-          <mesh filename="package://panther_description/meshes/components/rplidar_s1.stl" scale="0.0001 0.0001 0.0001" />
+          <mesh filename="package://panther_description/meshes/components/rplidar_a3.dae" scale="0.001 0.001 0.001" />
         </geometry>
-        <origin xyz="0 0 ${0.051/2}" rpy="0 0 -${pi/2}"/>
+        <origin xyz="0 0 0" rpy="${pi/2} 0 ${pi/2}"/>
         <material name="DarkGrey"/>
       </visual>
       <collision>
         <geometry>
-          <cylinder radius="${0.0555/2}" length="0.051" />
+          <cylinder radius="${0.0757/2}" length="0.0408" />
         </geometry>
-        <origin xyz="0 0 ${0.051/2}" rpy="0 0 0"/>
+        <origin xyz="0 0 0.0204" rpy="0 0 0"/>
       </collision>
       <inertial>
-        <mass value="0.105" />
+        <mass value="0.190" />
         <inertia ixx="1" ixy="0" ixz="0" iyy="1" iyz="0" izz="1" />
       </inertial>
     </link>
-    <link name="${prefix}_rplidar_s1_laser_link"></link>
-    <joint name="base_link_to_${prefix}_rplidar_s1_link_joint" type="fixed">
+    <link name="${prefix}_rplidar_a2_laser_link"></link>
+    <joint name="base_link_to_${prefix}_rplidar_a2_link_joint" type="fixed">
       <origin xyz="${xyz}" rpy="${rpy}" />
       <parent link="base_link" />
-      <child link="${prefix}_rplidar_s1_link" />
+      <child link="${prefix}_rplidar_a2_link" />
     </joint>
-    <joint name="${prefix}_rplidar_s1_laser_link_joint" type="fixed">
-      <origin xyz="0 0 0.04" rpy="0 0 0" />
-      <parent link="${prefix}_rplidar_s1_link" />
-      <child link="${prefix}_rplidar_s1_laser_link" />
+    <joint name="${prefix}_rplidar_a2_laser_link_joint" type="fixed">
+      <origin xyz="0 0 0.0308" rpy="0 0 0" />
+      <parent link="${prefix}_rplidar_a2_link" />
+      <child link="${prefix}_rplidar_a2_laser_link" />
     </joint>
-    <gazebo reference="${prefix}_rplidar_s1_link">
+    <gazebo reference="${prefix}_rplidar_a2_link">
       <material>Gazebo/DarkGrey</material>
     </gazebo>
-    <gazebo reference="${prefix}_rplidar_s1_laser_link">
-      <sensor type="${ray_type}" name="${prefix}_rplidar_s1_sensor">
-        <pose>0 0 0.04 0 0 0</pose>
+    <gazebo reference="${prefix}_rplidar_a2_laser_link">
+      <sensor type="${ray_type}" name="${prefix}_rplidar_a2_sensor">
+        <pose>0 0 0.0308 0 0 0</pose>
         <visualize>false</visualize>
         <update_rate>10</update_rate>
@@ -51,5 +51,5 @@
           <scan>
             <horizontal>
-              <samples>9200</samples>
+              <samples>400</samples>
               <resolution>1</resolution>
               <min_angle>-${pi}</min_angle>
@@ -58,17 +58,17 @@
           </scan>
           <range>
-            <min>0.1</min>
-            <max>40.0</max>
-            <resolution>0.03</resolution>
+            <min>0.2</min>
+            <max>16.0</max>
+            <resolution>0.08</resolution>
           </range>
           <noise>
             <type>gaussian</type>
-            <mean>0</mean>
-            <stddev>0.03</stddev>
+            <mean>0.05</mean>
+            <stddev>0.01</stddev>
           </noise>
         </ray>
         <plugin name="gazebo_ros_head_rplidar_controller" filename="${plugin_file_name}">
           <topicName>${topic}</topicName>
-          <frameName>${prefix}_rplidar_s1_laser_link</frameName>
+          <frameName>${prefix}_rplidar_a2_laser_link</frameName>
         </plugin>
       </sensor>

File: src/panther_description/urdf/components/rplidar_a3.gazebo.xacro (robot description, xacro)
@@ -1,5 +1,5 @@
 <?xml version="1.0"?>
 <robot xmlns:xacro="http://www.ros.org/wiki/xacro">
-  <xacro:macro name="rplidar_s1" params="xyz rpy use_gpu:=false prefix:=front topic:=laser/scan">
+  <xacro:macro name="rplidar_a3" params="xyz rpy use_gpu:=false prefix:=front topic:=laser/scan">
     <xacro:if value="${use_gpu}">
       <xacro:property name="ray_type" value="gpu_ray" />
@@ -10,40 +10,40 @@
       <xacro:property name="plugin_file_name" value="libgazebo_ros_laser.so" />
     </xacro:unless>
-    <link name="${prefix}_rplidar_s1_link">
+    <link name="${prefix}_rplidar_a3_link">
       <visual>
         <geometry>
-          <mesh filename="package://panther_description/meshes/components/rplidar_s1.stl" scale="0.0001 0.0001 0.0001" />
+          <mesh filename="package://panther_description/meshes/components/rplidar_a3.dae" scale="0.001 0.001 0.001" />
         </geometry>
-        <origin xyz="0 0 ${0.051/2}" rpy="0 0 -${pi/2}"/>
+        <origin xyz="0 0 0" rpy="${pi/2} 0 ${pi/2}"/>
         <material name="DarkGrey"/>
       </visual>
       <collision>
         <geometry>
-          <cylinder radius="${0.0555/2}" length="0.051" />
+          <cylinder radius="${0.0757/2}" length="0.0408" />
         </geometry>
-        <origin xyz="0 0 ${0.051/2}" rpy="0 0 0"/>
+        <origin xyz="0 0 0.0204" rpy="0 0 0"/>
       </collision>
       <inertial>
-        <mass value="0.105" />
+        <mass value="0.190" />
         <inertia ixx="1" ixy="0" ixz="0" iyy="1" iyz="0" izz="1" />
       </inertial>
     </link>
-    <link name="${prefix}_rplidar_s1_laser_link"></link>
-    <joint name="base_link_to_${prefix}_rplidar_s1_link_joint" type="fixed">
+    <link name="${prefix}_rplidar_a3_laser_link"></link>
+    <joint name="base_link_to_${prefix}_rplidar_a3_link_joint" type="fixed">
       <origin xyz="${xyz}" rpy="${rpy}" />
       <parent link="base_link" />
-      <child link="${prefix}_rplidar_s1_link" />
+      <child link="${prefix}_rplidar_a3_link" />
     </joint>
-    <joint name="${prefix}_rplidar_s1_laser_link_joint" type="fixed">
-      <origin xyz="0 0 0.04" rpy="0 0 0" />
-      <parent link="${prefix}_rplidar_s1_link" />
-      <child link="${prefix}_rplidar_s1_laser_link" />
+    <joint name="${prefix}_rplidar_a3_laser_link_joint" type="fixed">
+      <origin xyz="0 0 0.0308" rpy="0 0 0" />
+      <parent link="${prefix}_rplidar_a3_link" />
+      <child link="${prefix}_rplidar_a3_laser_link" />
     </joint>
-    <gazebo reference="${prefix}_rplidar_s1_link">
+    <gazebo reference="${prefix}_rplidar_a3_link">
       <material>Gazebo/DarkGrey</material>
     </gazebo>
-    <gazebo reference="${prefix}_rplidar_s1_laser_link">
-      <sensor type="${ray_type}" name="${prefix}_rplidar_s1_sensor">
-        <pose>0 0 0.04 0 0 0</pose>
+    <gazebo reference="${prefix}_rplidar_a3_laser_link">
+      <sensor type="${ray_type}" name="${prefix}_rplidar_a3_sensor">
+        <pose>0 0 0.0308 0 0 0</pose>
         <visualize>false</visualize>
         <update_rate>10</update_rate>
@@ -51,5 +51,5 @@
           <scan>
             <horizontal>
-              <samples>9200</samples>
+              <samples>1600</samples>
               <resolution>1</resolution>
               <min_angle>-${pi}</min_angle>
@@ -58,17 +58,17 @@
           </scan>
           <range>
-            <min>0.1</min>
-            <max>40.0</max>
-            <resolution>0.03</resolution>
+            <min>0.2</min>
+            <max>25.0</max>
+            <resolution>0.05</resolution>
           </range>
           <noise>
             <type>gaussian</type>
-            <mean>0</mean>
-            <stddev>0.03</stddev>
+            <mean>0.0</mean>
+            <stddev>0.01</stddev>
           </noise>
         </ray>
         <plugin name="gazebo_ros_head_rplidar_controller" filename="${plugin_file_name}">
           <topicName>${topic}</topicName>
-          <frameName>${prefix}_rplidar_s1_laser_link</frameName>
+          <frameName>${prefix}_rplidar_a3_laser_link</frameName>
         </plugin>
       </sensor>

File: src/panther_description/urdf/components/stereolabs_zed.gazebo.xacro (robot description, xacro)
@@ -1,5 +1,5 @@
 <?xml version="1.0"?>
 <robot xmlns:xacro="http://www.ros.org/wiki/xacro">
-  <xacro:macro name="rplidar_s1" params="xyz rpy use_gpu:=false prefix:=front topic:=laser/scan">
+  <xacro:macro name="stereolabs_zed" params="xyz rpy use_gpu:=false prefix:=front topic:=scan">
     <xacro:if value="${use_gpu}">
       <xacro:property name="ray_type" value="gpu_ray" />
@@ -10,8 +10,8 @@
       <xacro:property name="plugin_file_name" value="libgazebo_ros_laser.so" />
     </xacro:unless>
-    <link name="${prefix}_rplidar_s1_link">
+    <link name="${prefix}_stereolabs_zed_link">
       <visual>
         <geometry>
-          <mesh filename="package://panther_description/meshes/components/rplidar_s1.stl" scale="0.0001 0.0001 0.0001" />
+            <mesh filename="package://panther_description/meshes/components/stereolabs_zed.stl" scale="0.0001 0.0001 0.0001" />
         </geometry>
         <origin xyz="0 0 ${0.051/2}" rpy="0 0 -${pi/2}"/>
@@ -25,25 +25,19 @@
       </collision>
       <inertial>
-        <mass value="0.105" />
-        <inertia ixx="1" ixy="0" ixz="0" iyy="1" iyz="0" izz="1" />
+          <mass value="0.105" />
+          <inertia ixx="1" ixy="0" ixz="0" iyy="1" iyz="0" izz="1" />
       </inertial>
     </link>
-    <link name="${prefix}_rplidar_s1_laser_link"></link>
-    <joint name="base_link_to_${prefix}_rplidar_s1_link_joint" type="fixed">
+    <joint name="base_link_to_${prefix}_stereolabs_zed_link_joint" type="fixed">
       <origin xyz="${xyz}" rpy="${rpy}" />
       <parent link="base_link" />
-      <child link="${prefix}_rplidar_s1_link" />
+      <child link="${prefix}_stereolabs_zed_link" />
     </joint>
-    <joint name="${prefix}_rplidar_s1_laser_link_joint" type="fixed">
-      <origin xyz="0 0 0.04" rpy="0 0 0" />
-      <parent link="${prefix}_rplidar_s1_link" />
-      <child link="${prefix}_rplidar_s1_laser_link" />
-    </joint>
-    <gazebo reference="${prefix}_rplidar_s1_link">
+    <gazebo reference="${prefix}_stereolabs_zed_link">
       <material>Gazebo/DarkGrey</material>
     </gazebo>
-    <gazebo reference="${prefix}_rplidar_s1_laser_link">
-      <sensor type="${ray_type}" name="${prefix}_rplidar_s1_sensor">
-        <pose>0 0 0.04 0 0 0</pose>
+    <gazebo reference="${prefix}_stereolabs_zed_link">
+      <sensor type="${ray_type}" name="${prefix}_stereolabs_zed_sensor">
+        <pose>0 0 0.045 0 0 0</pose>
         <visualize>false</visualize>
         <update_rate>10</update_rate>
@@ -52,11 +46,11 @@
             <horizontal>
               <samples>9200</samples>
-              <resolution>1</resolution>
-              <min_angle>-${pi}</min_angle>
-              <max_angle>${pi}</max_angle>
+              <resolution>0.391</resolution>
+              <min_angle>-3.14159265</min_angle>
+              <max_angle>3.14159265</max_angle>
             </horizontal>
           </scan>
           <range>
-            <min>0.1</min>
+            <min>0.2</min>
             <max>40.0</max>
             <resolution>0.03</resolution>
@@ -64,11 +58,11 @@
           <noise>
             <type>gaussian</type>
-            <mean>0</mean>
-            <stddev>0.03</stddev>
+            <mean>0.05</mean>
+            <stddev>0.01</stddev>
           </noise>
         </ray>
         <plugin name="gazebo_ros_head_rplidar_controller" filename="${plugin_file_name}">
           <topicName>${topic}</topicName>
-          <frameName>${prefix}_rplidar_s1_laser_link</frameName>
+          <frameName>${prefix}_stereolabs_zed_link</frameName>
         </plugin>
       </sensor>

File: src/panther_description/urdf/components/velodyne_puck.gazebo.xacro (robot description, xacro)
@@ -1,5 +1,5 @@
 <?xml version="1.0"?>
 <robot xmlns:xacro="http://www.ros.org/wiki/xacro">
-  <xacro:macro name="rplidar_s1" params="xyz rpy use_gpu:=false prefix:=front topic:=laser/scan">
+  <xacro:macro name="velodyne_puck" params="xyz rpy use_gpu:=false prefix:=front topic:=laser/scan">
     <xacro:if value="${use_gpu}">
       <xacro:property name="ray_type" value="gpu_ray" />
@@ -10,40 +10,40 @@
       <xacro:property name="plugin_file_name" value="libgazebo_ros_laser.so" />
     </xacro:unless>
-    <link name="${prefix}_rplidar_s1_link">
+    <link name="${prefix}_velodyne_puck_link">
       <visual>
         <geometry>
-          <mesh filename="package://panther_description/meshes/components/rplidar_s1.stl" scale="0.0001 0.0001 0.0001" />
+          <mesh filename="package://panther_description/meshes/components/velodyne_puck.stl" scale="0.025035 0.025035 0.025035" />
         </geometry>
-        <origin xyz="0 0 ${0.051/2}" rpy="0 0 -${pi/2}"/>
+        <origin xyz="0 0 ${0.051/2}" rpy="${pi/2} 0 ${pi}"/>
         <material name="DarkGrey"/>
       </visual>
       <collision>
         <geometry>
-          <cylinder radius="${0.0555/2}" length="0.051" />
+          <cylinder radius="${0.090/2}" length="0.0717" />
         </geometry>
-        <origin xyz="0 0 ${0.051/2}" rpy="0 0 0"/>
+        <origin xyz="0 0 ${0.0717/2}" rpy="0 0 0"/>
       </collision>
       <inertial>
-        <mass value="0.105" />
+        <mass value="0.830" />
         <inertia ixx="1" ixy="0" ixz="0" iyy="1" iyz="0" izz="1" />
       </inertial>
     </link>
-    <link name="${prefix}_rplidar_s1_laser_link"></link>
-    <joint name="base_link_to_${prefix}_rplidar_s1_link_joint" type="fixed">
+    <link name="${prefix}_velodyne_puck_laser_link"></link>
+    <joint name="base_link_to_${prefix}_velodyne_puck_link_joint" type="fixed">
       <origin xyz="${xyz}" rpy="${rpy}" />
       <parent link="base_link" />
-      <child link="${prefix}_rplidar_s1_link" />
+      <child link="${prefix}_velodyne_puck_link" />
     </joint>
-    <joint name="${prefix}_rplidar_s1_laser_link_joint" type="fixed">
-      <origin xyz="0 0 0.04" rpy="0 0 0" />
-      <parent link="${prefix}_rplidar_s1_link" />
-      <child link="${prefix}_rplidar_s1_laser_link" />
+    <joint name="${prefix}_velodyne_puck_laser_link_joint" type="fixed">
+      <origin xyz="0 0 0.0378" rpy="0 0 0" />
+      <parent link="${prefix}_velodyne_puck_link" />
+      <child link="${prefix}_velodyne_puck_laser_link" />
     </joint>
-    <gazebo reference="${prefix}_rplidar_s1_link">
+    <gazebo reference="${prefix}_velodyne_puck_link">
       <material>Gazebo/DarkGrey</material>
     </gazebo>
-    <gazebo reference="${prefix}_rplidar_s1_laser_link">
-      <sensor type="${ray_type}" name="${prefix}_rplidar_s1_sensor">
-        <pose>0 0 0.04 0 0 0</pose>
+    <gazebo reference="${prefix}_velodyne_puck_laser_link">
+      <sensor type="${ray_type}" name="${prefix}_velodyne_puck_sensor">
+        <pose>0 0 0.0378 0 0 0</pose>
         <visualize>false</visualize>
         <update_rate>10</update_rate>
@@ -51,18 +51,24 @@
           <scan>
             <horizontal>
-              <samples>9200</samples>
+              <samples>3600</samples>
               <resolution>1</resolution>
               <min_angle>-${pi}</min_angle>
               <max_angle>${pi}</max_angle>
             </horizontal>
+            <vertical>
+              <samples>75</samples>
+              <resolution>1</resolution>
+              <min_angle>-${15/180*pi}</min_angle>
+              <max_angle>${15/180*pi}</max_angle>
+            </vertical>
           </scan>
           <range>
-            <min>0.1</min>
-            <max>40.0</max>
+            <min>0.2</min>
+            <max>100.0</max>
             <resolution>0.03</resolution>
           </range>
           <noise>
             <type>gaussian</type>
-            <mean>0</mean>
+            <mean>0.05</mean>
             <stddev>0.03</stddev>
           </noise>
@@ -70,5 +76,5 @@
         <plugin name="gazebo_ros_head_rplidar_controller" filename="${plugin_file_name}">
           <topicName>${topic}</topicName>
-          <frameName>${prefix}_rplidar_s1_laser_link</frameName>
+          <frameName>${prefix}_velodyne_puck_laser_link</frameName>
         </plugin>
       </sensor>

File: src/panther_description/urdf/gazebo_plugins.gazebo.xacro (robot description, xacro)
@@ -2,4 +2,9 @@
 <robot xmlns:xacro="http://www.ros.org/wiki/xacro">
   <xacro:include filename="$(find panther_description)/urdf/components/rplidar_s1.gazebo.xacro" />
+  <xacro:include filename="$(find panther_description)/urdf/components/rplidar_a2.gazebo.xacro" />
+  <xacro:include filename="$(find panther_description)/urdf/components/rplidar_a3.gazebo.xacro" />
+  <xacro:include filename="$(find panther_description)/urdf/components/velodyne_puck.gazebo.xacro" />
+  <xacro:include filename="$(find panther_description)/urdf/components/orbebec_astra.gazebo.xacro" />
+  <xacro:include filename="$(find panther_description)/urdf/components/ouster_os1_16.gazebo.xacro" />
   <xacro:macro name="wheel_driver" params="wheel_props common_props">
     <xacro:if value="${wheel_props['simulation']['driver'] == 'libgazebo_ros_skid_steer_drive'}">

File: src/panther_description/urdf/panther.urdf.xacro (robot description, xacro)
@@ -3,5 +3,5 @@
   <xacro:arg name="panther_common_props_path" default="$(find panther_description)/config/panther_common.yaml" />
   <xacro:arg name="wheel_props_path" default="$(find panther_description)/config/classic_wheels_props.yaml" />
-  <xacro:arg name="use_gpu" default="false" />
+  <xacro:arg name="use_gpu" default="true" />
   <!-- IMPORT YAML CONFIGS -->
   <xacro:property name="panther_common_props_file" value="$(arg panther_common_props_path)"  />
@@ -23,5 +23,5 @@
   <!-- GAZEBO PLUGINS -->
   <xacro:gazebo.wheel_driver wheel_props="${wheel_props}" common_props="${panther_common_props}" />
-  <xacro:gazebo.rplidar_s1 xyz="0.2 0 0.14" rpy="0 0 0" use_gpu="$(arg use_gpu)" />
+  <xacro:gazebo.rplidar_s1 xyz="0.2 0 0.2" rpy="0 0 0" use_gpu="true" />
   <gazebo>
     <plugin name="gazebo_ros_control" filename="libgazebo_ros_control.so">
