Commit message: Add IMU sensor | Match lidar noise with datasheets

File: src/panther_description/urdf/components/ouster_os1_32.gazebo.xacro (robot description, xacro)
@@ -13,15 +13,14 @@
       <visual>
         <geometry>
-          <!-- <mesh filename="package://panther_description/meshes/components/ouster_os1_32.stl" scale="0.0001 0.0001 0.0001" /> -->
-          <cylinder radius="${0.0555/2}" length="0.051" />
+          <mesh filename="package://panther_description/meshes/components/ouster_os1_32.stl" scale="1 1 0.65" />
         </geometry>
-        <origin xyz="0 0 ${0.051/2}" rpy="0 0 -${pi/2}"/>
-        <material name="DarkGrey"/>
+        <origin xyz="0 0 0" rpy="0 0 ${pi/2}"/>
+        <material name="Grey"/>
       </visual>
       <collision>
         <geometry>
-          <cylinder radius="${0.0555/2}" length="0.051" />
+          <cylinder radius="${0.0753/2}" length="0.0435" />
         </geometry>
-        <origin xyz="0 0 ${0.051/2}" rpy="0 0 0"/>
+        <origin xyz="0 0 ${0.0435/2}" rpy="0 0 0"/>
       </collision>
       <inertial>
@@ -37,10 +36,10 @@
     </joint>
     <joint name="${prefix}_ouster_os1_32_laser_link_joint" type="fixed">
-      <origin xyz="0 0 0.0378" rpy="0 0 0" />
+      <origin xyz="0 0 0.023" rpy="0 0 0" />
       <parent link="${prefix}_ouster_os1_32_link" />
       <child link="${prefix}_ouster_os1_32_laser_link" />
     </joint>
     <gazebo reference="${prefix}_ouster_os1_32_link">
-      <material>Gazebo/DarkGrey</material>
+      <material>Gazebo/Grey</material>
     </gazebo>
     <gazebo reference="${prefix}_ouster_os1_32_laser_link">
@@ -65,12 +64,12 @@
           </scan>
           <range>
-            <min>0.05</min>
-            <max>120.0</max>
-            <resolution>0.007</resolution>
+            <min>${0.0753/2+0.01}</min>
+            <max>100.0</max>
+            <resolution>0.003</resolution>
           </range>
           <noise>
             <type>gaussian</type>
             <mean>0.0</mean>
-            <stddev>0.007</stddev>
+            <stddev>0.008</stddev>
           </noise>
         </ray>

File: src/panther_description/urdf/components/rplidar_a2.gazebo.xacro (robot description, xacro)
@@ -60,10 +60,10 @@
             <min>0.2</min>
             <max>16.0</max>
-            <resolution>0.08</resolution>
+            <resolution>0.12</resolution>
           </range>
           <noise>
             <type>gaussian</type>
-            <mean>0.05</mean>
-            <stddev>0.01</stddev>
+            <mean>0.0</mean>
+            <stddev>0.026</stddev>
           </noise>
         </ray>

File: src/panther_description/urdf/components/rplidar_a3.gazebo.xacro (robot description, xacro)
@@ -60,10 +60,10 @@
             <min>0.2</min>
             <max>25.0</max>
-            <resolution>0.05</resolution>
+            <resolution>0.12</resolution>
           </range>
           <noise>
             <type>gaussian</type>
             <mean>0.0</mean>
-            <stddev>0.01</stddev>
+            <stddev>0.026</stddev>
           </noise>
         </ray>

File: src/panther_description/urdf/components/rplidar_s1.gazebo.xacro (robot description, xacro)
@@ -58,12 +58,12 @@
           </scan>
           <range>
-            <min>0.1</min>
+            <min>${0.051/2+0.001}</min>
             <max>40.0</max>
-            <resolution>0.015</resolution>
+            <resolution>0.03</resolution>
           </range>
           <noise>
             <type>gaussian</type>
             <mean>0</mean>
-            <stddev>0.00125</stddev>
+            <stddev>0.026</stddev>
           </noise>
         </ray>

File: src/panther_description/urdf/components/velodyne_puck.gazebo.xacro (robot description, xacro)
@@ -15,5 +15,5 @@
           <mesh filename="package://panther_description/meshes/components/velodyne_puck.stl" scale="0.025035 0.025035 0.025035" />
         </geometry>
-        <origin xyz="0 0 ${0.051/2}" rpy="${pi/2} 0 ${pi}"/>
+        <origin xyz="0 0 0" rpy="${pi/2} 0 ${pi}"/>
         <material name="DarkGrey"/>
       </visual>
@@ -64,12 +64,12 @@
           </scan>
           <range>
-            <min>0.2</min>
+            <min>${0.051+0.01}</min>
             <max>100.0</max>
-            <resolution>0.015</resolution>
+            <resolution>0.005</resolution>
           </range>
           <noise>
             <type>gaussian</type>
-            <mean>0.05</mean>
-            <stddev>0.03</stddev>
+            <mean>0.0</mean>
+            <stddev>0.016</stddev>
           </noise>
         </ray>

File: src/panther_description/urdf/gazebo_plugins.gazebo.xacro (robot description, xacro)
@@ -43,4 +43,35 @@
       </gazebo>
     </xacro:if>
+    <link name="imu">
+      <inertial>
+        <mass value="0.0000001" />
+        <inertia ixx="1" ixy="0" ixz="0" iyy="1" iyz="0" izz="1" />
+      </inertial>
+    </link>
+    <joint name="base_link_to_imu_link_joint" type="fixed">
+      <origin xyz="0.169 0.025 0.092" rpy="0 0 0" />
+      <parent link="base_link" />
+      <child link="imu" />
+    </joint>
+    <gazebo reference="imu">
+      <gravity>true</gravity>
+      <sensor name="imu_sensor" type="imu">
+        <always_on>true</always_on>
+        <update_rate>100</update_rate>
+        <visualize>false</visualize>
+        <topic>imu/data</topic>
+        <plugin filename="libgazebo_ros_imu_sensor.so" name="imu_plugin">
+          <topicName>imu/data</topicName>
+          <bodyName>imu</bodyName>
+          <updateRateHZ>125.0</updateRateHZ>
+          <gaussianNoise>${0.095*(pi/180.0)}</gaussianNoise>
+          <xyzOffset>0 0 0</xyzOffset>
+          <rpyOffset>0 0 0</rpyOffset>
+          <frameName>imu</frameName>
+          <initialOrientationAsReference>false</initialOrientationAsReference>
+        </plugin>
+        <pose>0 0 0 0 0 0</pose>
+      </sensor>
+    </gazebo>
   </xacro:macro>
 </robot>

File: src/panther_description/urdf/panther.urdf.xacro (robot description, xacro)
@@ -3,5 +3,5 @@
   <xacro:arg name="panther_common_props_path" default="$(find panther_description)/config/panther_common.yaml" />
   <xacro:arg name="wheel_props_path" default="$(find panther_description)/config/classic_wheels_props.yaml" />
-  <xacro:arg name="use_gpu" default="false" />
+  <xacro:arg name="use_gpu" default="true" />
   <!-- IMPORT YAML CONFIGS -->
   <xacro:property name="panther_common_props_file" value="$(arg panther_common_props_path)"  />
@@ -23,5 +23,5 @@
   <!-- GAZEBO PLUGINS -->
   <xacro:gazebo.wheel_driver wheel_props="${wheel_props}" common_props="${panther_common_props}" />
-  <xacro:gazebo.rplidar_s1 xyz="0.185 0 0.17" rpy="0 0 0" use_gpu="$(arg use_gpu)" />
+  <xacro:gazebo.rplidar_a3 xyz="0.185 0 0.17" rpy="0 0 0" use_gpu="$(arg use_gpu)" />
   <gazebo>
     <plugin name="gazebo_ros_control" filename="libgazebo_ros_control.so">
