Commit message: Update wheels names | Fix typo

File: panther_description/urdf/components/orbbec_astra.gazebo.xacro (robot description, xacro)
@@ -5,5 +5,5 @@
       <visual>
         <geometry>
-            <mesh filename="package://panther_description/meshes/components/orbbec_astra.dae" scale="0.001 0.001 0.001" />
+            <mesh filename="package://panther_description/meshes/components/orbbec_astra.stl" scale="0.001 0.001 0.001" />
         </geometry>
         <origin xyz="-0.01 0 0.025" rpy="${pi/2} 0 ${pi/2}"/>
