Commit message: Fix base_link location

File: panther_description/models/panther/body.urdf.xacro (robot description, xacro)
@@ -2,5 +2,5 @@
 <robot xmlns:xacro="http://www.ros.org/wiki/xacro">
   <!-- body defining macro -->
-  <xacro:macro name="body" params="props">
+  <xacro:macro name="body" params="props wheel_props">
     <link name="base_link"></link>
     <link name="body_link">
@@ -71,5 +71,5 @@
     </link>
     <joint name="base_link_to_body_joint" type="fixed">
-      <origin xyz="0 0 0" rpy="0 0 0" />
+      <origin xyz="0 0 ${wheel_props['diameter']/2}" rpy="0 0 0" />
       <parent link="base_link" />
       <child link="body_link" />
@@ -85,12 +85,12 @@
       <child link="rails_link" />
     </joint>
-    <joint name="base_link_to_imu_link_joint" type="fixed">
+    <joint name="body_link_to_imu_link_joint" type="fixed">
       <origin xyz="0.169 0.025 0.092" rpy="0 0 0" />
-      <parent link="base_link" />
+      <parent link="body_link" />
       <child link="imu_link" />
     </joint>
-    <joint name="base_link_to_gps_link_joint" type="fixed">
+    <joint name="body_link_to_gps_link_joint" type="fixed">
       <origin xyz="0.169 0.025 0.092" rpy="0 0 0" />
-      <parent link="base_link" />
+      <parent link="body_link" />
       <child link="gps_link" />
     </joint>

File: panther_description/models/panther/components/orbbec_astra.gazebo.xacro (robot description, xacro)
@@ -23,7 +23,7 @@
     <link name="${prefix}_orbbec_astra_depth_link"></link>
     <link name="${prefix}_orbbec_astra_depth_refference_link"></link>
-    <joint name="base_link_to_${prefix}_orbbec_astra_link_joint" type="fixed">
+    <joint name="body_link_to_${prefix}_orbbec_astra_link_joint" type="fixed">
       <origin xyz="${xyz}" rpy="${rpy}" />
-      <parent link="base_link" />
+      <parent link="body_link" />
       <child link="${prefix}_orbbec_astra_link" />
     </joint>

File: panther_description/models/panther/components/ouster_os1_32.gazebo.xacro (robot description, xacro)
@@ -30,7 +30,7 @@
     </link>
     <link name="${prefix}_ouster_os1_32_laser_link"></link>
-    <joint name="base_link_to_${prefix}_ouster_os1_32_link_joint" type="fixed">
+    <joint name="body_link_to_${prefix}_ouster_os1_32_link_joint" type="fixed">
       <origin xyz="${xyz}" rpy="${rpy}" />
-      <parent link="base_link" />
+      <parent link="body_link" />
       <child link="${prefix}_ouster_os1_32_link" />
     </joint>

File: panther_description/models/panther/components/rplidar_s1.gazebo.xacro (robot description, xacro)
@@ -28,7 +28,7 @@
     </link>
     <link name="${prefix}_rplidar_s1_laser_link"></link>
-    <joint name="base_link_to_${prefix}_rplidar_s1_link_joint" type="fixed">
+    <joint name="body_link_to_${prefix}_rplidar_s1_link_joint" type="fixed">
       <origin xyz="${xyz}" rpy="${rpy}" />
-      <parent link="base_link" />
+      <parent link="body_link" />
       <child link="${prefix}_rplidar_s1_link" />
     </joint>

File: panther_description/models/panther/components/velodyne_puck.gazebo.xacro (robot description, xacro)
@@ -28,7 +28,7 @@
     </link>
     <link name="${prefix}_velodyne_puck_laser_link"></link>
-    <joint name="base_link_to_${prefix}_velodyne_puck_link_joint" type="fixed">
+    <joint name="body_link_to_${prefix}_velodyne_puck_link_joint" type="fixed">
       <origin xyz="${xyz}" rpy="${rpy}" />
-      <parent link="base_link" />
+      <parent link="body_link" />
       <child link="${prefix}_velodyne_puck_link" />
     </joint>

File: panther_description/models/panther/gazebo_plugins.gazebo.xacro (robot description, xacro)
@@ -11,23 +11,16 @@
           <ros>
           </ros>
-          <!-- Update rate -->
           <update_rate>10</update_rate>
-          <!-- Number of wheel pairs -->
           <num_wheel_pairs>2</num_wheel_pairs>
-          <!-- wheels0 -->
           <left_joint>front_left_wheel_joint</left_joint>
           <right_joint>front_right_wheel_joint</right_joint>
-          <!-- wheels1-->
           <left_joint>rear_left_wheel_joint</left_joint>
           <right_joint>rear_right_wheel_joint</right_joint>
-          <!-- kinematics -->
           <wheel_separation>${wheel_props['wheels']['wheel_separation']}</wheel_separation>
           <wheel_separation>${wheel_props['wheels']['wheel_separation']}</wheel_separation>
           <wheel_diameter>${wheel_props['wheels']['diameter']}</wheel_diameter>
           <wheel_diameter>${wheel_props['wheels']['diameter']}</wheel_diameter>
-          <!-- limits -->
           <max_wheel_torque>${common_props['motors']['max_torque']}</max_wheel_torque>
           <max_wheel_acceleration>2.0</max_wheel_acceleration>
-          <!-- output -->
           <publish_odom>true</publish_odom>
           <publish_odom_tf>true</publish_odom_tf>
@@ -43,15 +36,10 @@
           <ros>
           </ros>
-          <!-- Set control loop update rate -->
-          <update_rate>100</update_rate>
-          <!-- Set odom publish rate -->
+          <update_rate>10</update_rate>
           <publish_rate>10</publish_rate>
-          <!-- Set if odom required -->
           <publish_odom>true</publish_odom>
           <publish_odom_tf>true</publish_odom_tf>
-          <!-- Frame IDs -->
           <odometry_frame>odom</odometry_frame>
           <robot_base_frame>base_link</robot_base_frame>
-          <!-- Set odom covariance -->
           <covariance_x>0.0001</covariance_x>
           <covariance_y>0.0001</covariance_y>

File: panther_description/models/panther/panther.urdf.xacro (robot description, xacro)
@@ -15,5 +15,5 @@
   <xacro:include filename="$(find panther_description)/models/panther/gazebo_plugins.gazebo.xacro" ns="gazebo" />
   <!-- BODY DECLARATION -->
-  <xacro:body.body props="${panther_common_props['body']}" />
+  <xacro:body.body props="${panther_common_props['body']}" wheel_props="${wheel_props['wheels']}" />
   <!-- WHEEL DECLARATION -->
   <xacro:wheel.wheel wheel_props="${wheel_props['wheels']}" common_props="${panther_common_props}" prefix="front_left" />
