Commit message: base_link between wheel | 3d lidar as pointcloud

File: panther_description/urdf/body.urdf.xacro (robot description, xacro)
@@ -2,5 +2,5 @@
 <robot xmlns:xacro="http://www.ros.org/wiki/xacro">
   <!-- body defining macro -->
-  <xacro:macro name="body" params="props">
+  <xacro:macro name="body" params="props wheel_props">
     <link name="base_link"></link>
     <link name="body_link">
@@ -71,5 +71,5 @@
     </link>
     <joint name="base_link_to_body_joint" type="fixed">
-      <origin xyz="0 0 0" rpy="0 0 0" />
+      <origin xyz="0 0 ${wheel_props['diameter']/2}" rpy="0 0 0" />
       <parent link="base_link" />
       <child link="body_link" />
@@ -85,12 +85,12 @@
       <child link="rails_link" />
     </joint>
-    <joint name="base_link_to_imu_link_joint" type="fixed">
+    <joint name="body_link_to_imu_link_joint" type="fixed">
       <origin xyz="0.169 0.025 0.092" rpy="0 0 0" />
-      <parent link="base_link" />
+      <parent link="body_link" />
       <child link="imu_link" />
     </joint>
-    <joint name="base_link_to_gps_link_joint" type="fixed">
+    <joint name="body_link_to_gps_link_joint" type="fixed">
       <origin xyz="0.169 0.025 0.092" rpy="0 0 0" />
-      <parent link="base_link" />
+      <parent link="body_link" />
       <child link="gps_link" />
     </joint>

File: panther_description/urdf/components/orbbec_astra.gazebo.xacro (robot description, xacro)
@@ -22,7 +22,7 @@
     </link>
     <link name="${prefix}_orbbec_astra_depth_link"></link>
-    <joint name="base_link_to_${prefix}_orbbec_astra_link_joint" type="fixed">
+    <joint name="body_link_to_${prefix}_orbbec_astra_link_joint" type="fixed">
       <origin xyz="${xyz}" rpy="${rpy}" />
-      <parent link="base_link" />
+      <parent link="body_link" />
       <child link="${prefix}_orbbec_astra_link" />
     </joint>

File: panther_description/urdf/components/ouster_os1_32.gazebo.xacro (robot description, xacro)
@@ -30,7 +30,7 @@
     </link>
     <link name="${prefix}_ouster_os1_32_laser_link"></link>
-    <joint name="base_link_to_${prefix}_ouster_os1_32_link_joint" type="fixed">
+    <joint name="body_link_to_${prefix}_ouster_os1_32_link_joint" type="fixed">
       <origin xyz="${xyz}" rpy="${rpy}" />
-      <parent link="base_link" />
+      <parent link="body_link" />
       <child link="${prefix}_ouster_os1_32_link" />
     </joint>
@@ -44,5 +44,5 @@
     </gazebo>
     <gazebo reference="${prefix}_ouster_os1_32_laser_link">
-      <sensor type="${ray_type}" name="${prefix}_ouster_os1_32_sensor">
+      <sensor type="ray" name="${prefix}_ouster_os1_32_sensor">
         <pose>0 0 0.0 0 0 0</pose>
         <visualize>false</visualize>
@@ -74,7 +74,9 @@
           </noise>
         </ray>
-        <plugin name="gazebo_ros_head_rplidar_controller" filename="${plugin_file_name}">
+        <plugin name="gazebo_ros_block_laser_controller" filename="libgazebo_ros_block_laser.so">
           <topicName>${topic}</topicName>
           <frameName>${prefix}_ouster_os1_32_laser_link</frameName>
+          <gaussianNoise>0.0008</gaussianNoise>
+          <updateRate>10</updateRate>
         </plugin>
       </sensor>

File: panther_description/urdf/components/rplidar_s1.gazebo.xacro (robot description, xacro)
@@ -30,7 +30,7 @@
     </link>
     <link name="${prefix}_rplidar_s1_laser_link"></link>
-    <joint name="base_link_to_${prefix}_rplidar_s1_link_joint" type="fixed">
+    <joint name="body_link_to_${prefix}_rplidar_s1_link_joint" type="fixed">
       <origin xyz="${xyz}" rpy="${rpy}" />
-      <parent link="base_link" />
+      <parent link="body_link" />
       <child link="${prefix}_rplidar_s1_link" />
     </joint>

File: panther_description/urdf/components/velodyne_puck.gazebo.xacro (robot description, xacro)
@@ -2,12 +2,4 @@
 <robot xmlns:xacro="http://www.ros.org/wiki/xacro">
   <xacro:macro name="velodyne_puck" params="xyz rpy use_gpu:=false prefix:=front topic:=laser/scan">
-    <xacro:if value="${use_gpu}">
-      <xacro:property name="ray_type" value="gpu_ray" />
-      <xacro:property name="plugin_file_name" value="libgazebo_ros_gpu_laser.so" />
-    </xacro:if>
-    <xacro:unless value="${use_gpu}">
-      <xacro:property name="ray_type" value="ray" />
-      <xacro:property name="plugin_file_name" value="libgazebo_ros_laser.so" />
-    </xacro:unless>
     <link name="${prefix}_velodyne_puck_link">
       <visual>
@@ -30,7 +22,7 @@
     </link>
     <link name="${prefix}_velodyne_puck_laser_link"></link>
-    <joint name="base_link_to_${prefix}_velodyne_puck_link_joint" type="fixed">
+    <joint name="body_link_to_${prefix}_velodyne_puck_link_joint" type="fixed">
       <origin xyz="${xyz}" rpy="${rpy}" />
-      <parent link="base_link" />
+      <parent link="body_link" />
       <child link="${prefix}_velodyne_puck_link" />
     </joint>
@@ -44,5 +36,5 @@
     </gazebo>
     <gazebo reference="${prefix}_velodyne_puck_laser_link">
-      <sensor type="${ray_type}" name="${prefix}_velodyne_puck_sensor">
+      <sensor type="ray" name="${prefix}_velodyne_puck_sensor">
         <pose>0 0 0.0378 0 0 0</pose>
         <visualize>false</visualize>
@@ -74,7 +66,9 @@
           </noise>
         </ray>
-        <plugin name="gazebo_ros_head_rplidar_controller" filename="${plugin_file_name}">
+        <plugin name="gazebo_ros_block_laser_controller" filename="libgazebo_ros_block_laser.so">
           <topicName>${topic}</topicName>
           <frameName>${prefix}_velodyne_puck_laser_link</frameName>
+          <gaussianNoise>0.0008</gaussianNoise>
+          <updateRate>10</updateRate>
         </plugin>
       </sensor>

File: panther_description/urdf/panther.urdf.xacro (robot description, xacro)
@@ -15,5 +15,5 @@
   <xacro:include filename="$(find panther_description)/urdf/gazebo_plugins.gazebo.xacro" ns="gazebo" />
   <!-- BODY DECLARATION -->
-  <xacro:body.body props="${panther_common_props['body']}" />
+  <xacro:body.body props="${panther_common_props['body']}" wheel_props="${wheel_props['wheels']}" />
   <!-- WHEEL DECLARATION -->
   <xacro:wheel.wheel wheel_props="${wheel_props['wheels']}" common_props="${panther_common_props}" prefix="front_left" />
