Commit message: Update meshes and package.xml

File: urdf/components/external_antenna.urdf.xacro (robot description, xacro)
@@ -26,5 +26,5 @@
       <collision>
         <geometry>
-          <mesh filename="file://$(find panther_description)/meshes/components/external_antenna.dae" />
+          <mesh filename="file://$(find panther_description)/meshes/components/external_antenna_collision.stl" />
         </geometry>
         <origin xyz="0.0 0.0 0.0" rpy="0.0 0.0 0.0"/>
