Commit message: Add support for ROS 2

File: examples/dual_rplidar_s1_and_orbbec_asta/panther.urdf.xacro (robot description, xacro)
@@ -26,9 +26,3 @@
   <xacro:gazebo.rplidar_s1 xyz="-0.185 0 0.17" rpy="0 0 ${pi/2}" use_gpu="$(arg use_gpu)" prefix="rear" topic="laser/rear/scan" />
   <xacro:gazebo.orbbec_astra xyz="0.36 0 0.025" rpy="0 0 0" />
-  <gazebo>
-    <plugin name="gazebo_ros_control" filename="libgazebo_ros_control.so">
-      <robotNamespace>/</robotNamespace>
-      <legacyModeNS>true</legacyModeNS>
-    </plugin>
-  </gazebo>
 </robot>

File: examples/ouster_os1_32/panther.urdf.xacro (robot description, xacro)
@@ -24,9 +24,3 @@
   <xacro:gazebo.wheel_driver wheel_props="${wheel_props}" common_props="${panther_common_props}" />
   <xacro:gazebo.ouster_os1_32 xyz="0.185 0 0.17" rpy="0 0 0" use_gpu="$(arg use_gpu)" />
-  <gazebo>
-    <plugin name="gazebo_ros_control" filename="libgazebo_ros_control.so">
-      <robotNamespace>/</robotNamespace>
-      <legacyModeNS>true</legacyModeNS>
-    </plugin>
-  </gazebo>
 </robot>

File: panther_description/models/panther/body.urdf.xacro (robot description, xacro)
@@ -8,5 +8,5 @@
         <geometry>
             <xacro:property name="mesh" value="${props['visual']['base']['mesh']}" />
-            <mesh filename="package://panther_description/meshes/${mesh}" scale="1 1 1" />
+            <mesh filename="file://$(find panther_description)/models/panther//meshes/${mesh}" scale="1 1 1" />
         </geometry>
         <origin xyz="0 0 0" rpy=" ${pi/2} 0 ${pi/2}"/>
@@ -16,5 +16,5 @@
         <geometry>
             <xacro:property name="mesh" value="${props['collision']['mesh']}" />
-            <mesh filename="package://panther_description/meshes/${mesh}" scale="1 1 1" />
+            <mesh filename="file://$(find panther_description)/models/panther//meshes/${mesh}" scale="1 1 1" />
         </geometry>
         <origin xyz="0 0 0" rpy=" ${pi/2} 0 ${pi/2}"/>
@@ -38,5 +38,5 @@
         <geometry>
           <xacro:property name="mesh" value="${props['visual']['cover']['mesh']}" />
-          <mesh filename="package://panther_description/meshes/${mesh}" scale="1 1 1" />
+          <mesh filename="file://$(find panther_description)/models/panther/meshes/${mesh}" scale="1 1 1" />
         </geometry>
         <origin xyz="0 0 0" rpy=" ${pi/2} 0 ${pi/2}"/>
@@ -52,5 +52,5 @@
         <geometry>
           <xacro:property name="mesh" value="${props['visual']['rails']['mesh']}" />
-          <mesh filename="package://panther_description/meshes/${mesh}" scale="1 1 1" />
+          <mesh filename="file://$(find panther_description)/models/panther//meshes/${mesh}" scale="1 1 1" />
         </geometry>
         <origin xyz="0 0 0" rpy=" ${pi/2} 0 ${pi/2}"/>

File: panther_description/models/panther/components/ouster_os1_32.gazebo.xacro (robot description, xacro)
@@ -4,14 +4,14 @@
     <xacro:if value="${use_gpu}">
       <xacro:property name="ray_type" value="gpu_ray" />
-      <xacro:property name="plugin_file_name" value="libgazebo_ros_gpu_laser.so" />
+      <xacro:property name="plugin_file_name" value="libgazebo_ros_gpu_ray_sensor.so" />
     </xacro:if>
     <xacro:unless value="${use_gpu}">
       <xacro:property name="ray_type" value="ray" />
-      <xacro:property name="plugin_file_name" value="libgazebo_ros_laser.so" />
+      <xacro:property name="plugin_file_name" value="libgazebo_ros_ray_sensor.so" />
     </xacro:unless>
     <link name="${prefix}_ouster_os1_32_link">
       <visual>
         <geometry>
-          <mesh filename="package://panther_description/meshes/components/ouster_os1_32.stl" scale="1 1 0.65" />
+          <mesh filename="file://$(find panther_description)/models/panther/meshes/components/ouster_os1_32.stl" scale="1 1 0.65" />
         </geometry>
         <origin xyz="0 0 0" rpy="0 0 ${pi/2}"/>
@@ -44,8 +44,7 @@
     </gazebo>
     <gazebo reference="${prefix}_ouster_os1_32_laser_link">
-      <sensor type="${ray_type}" name="${prefix}_ouster_os1_32_sensor">
+      <sensor type="${ray_type}" name="${prefix}_velodyne_puck_sensor">
         <pose>0 0 0.0 0 0 0</pose>
         <visualize>false</visualize>
-        <update_rate>10</update_rate>
         <ray>
           <scan>
@@ -74,7 +73,12 @@
           </noise>
         </ray>
-        <plugin name="gazebo_ros_head_rplidar_controller" filename="${plugin_file_name}">
-          <topicName>${topic}</topicName>
-          <frameName>${prefix}_ouster_os1_32_laser_link</frameName>
+        <update_rate>10</update_rate>
+        <plugin name="scan" filename="libgazebo_ros_ray_sensor.so">
+          <ros>
+            <namespace>/</namespace>
+            <argument>~/out:=${topic}</argument>
+          </ros>
+          <output_type>sensor_msgs/PointCloud2</output_type>
+          <frame_name>${prefix}_ouster_os1_32_laser_link</frame_name>
         </plugin>
       </sensor>

File: panther_description/models/panther/components/rplidar_s1.gazebo.xacro (robot description, xacro)
@@ -4,14 +4,12 @@
     <xacro:if value="${use_gpu}">
       <xacro:property name="ray_type" value="gpu_ray" />
-      <xacro:property name="plugin_file_name" value="libgazebo_ros_gpu_laser.so" />
     </xacro:if>
     <xacro:unless value="${use_gpu}">
       <xacro:property name="ray_type" value="ray" />
-      <xacro:property name="plugin_file_name" value="libgazebo_ros_laser.so" />
     </xacro:unless>
     <link name="${prefix}_rplidar_s1_link">
       <visual>
         <geometry>
-          <mesh filename="package://panther_description/meshes/components/rplidar_s1.stl" scale="0.0001 0.0001 0.0001" />
+          <mesh filename="file://$(find panther_description)/models/panther/meshes/components/rplidar_s1.stl" scale="0.0001 0.0001 0.0001" />
         </geometry>
         <origin xyz="0 0 ${0.051/2}" rpy="0 0 -${pi/2}"/>
@@ -47,5 +45,4 @@
         <pose>0 0 0.04 0 0 0</pose>
         <visualize>false</visualize>
-        <update_rate>10</update_rate>
         <ray>
           <scan>
@@ -64,11 +61,16 @@
           <noise>
             <type>gaussian</type>
-            <mean>0</mean>
+            <mean>0.0</mean>
             <stddev>0.001</stddev>
           </noise>
         </ray>
-        <plugin name="gazebo_ros_head_rplidar_controller" filename="${plugin_file_name}">
-          <topicName>${topic}</topicName>
-          <frameName>${prefix}_rplidar_s1_laser_link</frameName>
+        <update_rate>10</update_rate>
+        <plugin name="scan" filename="libgazebo_ros_ray_sensor.so">
+          <ros>
+            <namespace>/</namespace>
+            <argument>~/out:=${topic}</argument>
+          </ros>
+          <output_type>sensor_msgs/LaserScan</output_type>
+          <frame_name>${prefix}_rplidar_s1_laser_link</frame_name>
         </plugin>
       </sensor>

File: panther_description/models/panther/components/velodyne_puck.gazebo.xacro (robot description, xacro)
@@ -4,14 +4,12 @@
     <xacro:if value="${use_gpu}">
       <xacro:property name="ray_type" value="gpu_ray" />
-      <xacro:property name="plugin_file_name" value="libgazebo_ros_gpu_laser.so" />
     </xacro:if>
     <xacro:unless value="${use_gpu}">
       <xacro:property name="ray_type" value="ray" />
-      <xacro:property name="plugin_file_name" value="libgazebo_ros_laser.so" />
     </xacro:unless>
     <link name="${prefix}_velodyne_puck_link">
       <visual>
         <geometry>
-          <mesh filename="package://panther_description/meshes/components/velodyne_puck.stl" scale="0.025035 0.025035 0.025035" />
+          <mesh filename="file://$(find panther_description)/models/panther/meshes/components/velodyne_puck.stl" scale="0.025035 0.025035 0.025035" />
         </geometry>
         <origin xyz="0 0 0" rpy="${pi/2} 0 ${pi}"/>
@@ -47,5 +45,4 @@
         <pose>0 0 0.0378 0 0 0</pose>
         <visualize>false</visualize>
-        <update_rate>10</update_rate>
         <ray>
           <scan>
@@ -74,7 +71,12 @@
           </noise>
         </ray>
-        <plugin name="gazebo_ros_head_rplidar_controller" filename="${plugin_file_name}">
-          <topicName>${topic}</topicName>
-          <frameName>${prefix}_velodyne_puck_laser_link</frameName>
+        <update_rate>10</update_rate>
+        <plugin name="scan" filename="libgazebo_ros_ray_sensor.so">
+          <ros>
+            <namespace>/</namespace>
+            <argument>~/out:=${topic}</argument>
+          </ros>
+          <output_type>sensor_msgs/PointCloud2</output_type>
+          <frame_name>${prefix}_velodyne_puck_laser_link</frame_name>
         </plugin>
       </sensor>

File: panther_description/models/panther/panther.urdf.xacro (robot description, xacro)
@@ -1,7 +1,7 @@
 <?xml version='1.0'?>
 <robot name="panther" xmlns:xacro="http://www.ros.org/wiki/xacro">
-  <xacro:arg name="panther_common_props_path" default="$(find panther_description)/config/panther_common.yaml" />
-  <xacro:arg name="wheel_props_path" default="$(find panther_description)/config/WH01.yaml" />
-  <xacro:arg name="use_gpu" default="false" />
+  <xacro:arg name="panther_common_props_path" default="$(find panther_description)/models/panther/config/panther_common.yaml" />
+  <xacro:arg name="wheel_props_path" default="$(find panther_description)/models/panther/config/WH01.yaml" />
+  <xacro:arg name="use_gpu" default="true" />
   <!-- IMPORT YAML CONFIGS -->
   <xacro:property name="panther_common_props_file" value="$(arg panther_common_props_path)"  />
@@ -10,8 +10,8 @@
   <xacro:property name="wheel_props" value="${load_yaml(wheel_props_file)}" />
   <!-- INCLUDE ROBOT PARTS DEFINITIONS -->
-  <xacro:include filename="$(find panther_description)/urdf/materials.urdf.xacro" />
-  <xacro:include filename="$(find panther_description)/urdf/body.urdf.xacro" ns="body" />
-  <xacro:include filename="$(find panther_description)/urdf/wheel.urdf.xacro" ns="wheel" />
-  <xacro:include filename="$(find panther_description)/urdf/gazebo_plugins.gazebo.xacro" ns="gazebo" />
+  <xacro:include filename="$(find panther_description)/models/panther/materials.urdf.xacro" />
+  <xacro:include filename="$(find panther_description)/models/panther/body.urdf.xacro" ns="body" />
+  <xacro:include filename="$(find panther_description)/models/panther/wheel.urdf.xacro" ns="wheel" />
+  <xacro:include filename="$(find panther_description)/models/panther/gazebo_plugins.gazebo.xacro" ns="gazebo" />
   <!-- BODY DECLARATION -->
   <xacro:body.body props="${panther_common_props['body']}" />
@@ -24,9 +24,3 @@
   <xacro:gazebo.wheel_driver wheel_props="${wheel_props}" common_props="${panther_common_props}" />
   <xacro:gazebo.rplidar_s1 xyz="0.185 0 0.17" rpy="0 0 0" use_gpu="$(arg use_gpu)" />
-  <gazebo>
-    <plugin name="gazebo_ros_control" filename="libgazebo_ros_control.so">
-      <robotNamespace>/</robotNamespace>
-      <legacyModeNS>true</legacyModeNS>
-    </plugin>
-  </gazebo>
 </robot>

File: panther_description/models/panther/wheel.urdf.xacro (robot description, xacro)
@@ -8,20 +8,20 @@
       <xacro:property name="x" value="0.22" />
       <xacro:property name="y" value="${wheel_props['wheel_separation']/2}" />
-      <xacro:property name="mesh" value="package://panther_description/meshes/${mesh_folder}/wheel_a.stl" />
+      <xacro:property name="mesh" value="file://$(find panther_description)/models/panther/meshes/${mesh_folder}/wheel_a.stl" />
     </xacro:if>
     <xacro:if value="${prefix == 'front_right'}">
       <xacro:property name="x" value="0.22" />
       <xacro:property name="y" value="-${wheel_props['wheel_separation']/2}" />
-      <xacro:property name="mesh" value="package://panther_description/meshes/${mesh_folder}/wheel_b.stl" />
+      <xacro:property name="mesh" value="file://$(find panther_description)/models/panther/meshes/${mesh_folder}/wheel_b.stl" />
     </xacro:if>
     <xacro:if value="${prefix == 'rear_left'}">
       <xacro:property name="x" value="-0.22" />
       <xacro:property name="y" value="${wheel_props['wheel_separation']/2}" />
-      <xacro:property name="mesh" value="package://panther_description/meshes/${mesh_folder}/wheel_a.stl" />
+      <xacro:property name="mesh" value="file://$(find panther_description)/models/panther/meshes/${mesh_folder}/wheel_a.stl" />
     </xacro:if>
     <xacro:if value="${prefix == 'rear_right'}">
       <xacro:property name="x" value="-0.22" />
       <xacro:property name="y" value="-${wheel_props['wheel_separation']/2}" />
-      <xacro:property name="mesh" value="package://panther_description/meshes/${mesh_folder}/wheel_b.stl" />
+      <xacro:property name="mesh" value="file://$(find panther_description)/models/panther/meshes/${mesh_folder}/wheel_b.stl" />
     </xacro:if>
     <link name="${prefix}_wheel_link">
@@ -35,5 +35,5 @@
       <collision>
         <geometry>
-            <mesh filename="package://panther_description/meshes/${mesh_folder}/collision.stl" scale="1 1 1" />
+            <mesh filename="file://$(find panther_description)/models/panther/meshes/${mesh_folder}/collision.stl" scale="1 1 1" />
         </geometry>
         <origin xyz="0 0 0" rpy="${rpy}" />
@@ -59,14 +59,4 @@
                 friction="${common_props['motors']['joint_friction']}"/>
     </joint>
-    <transmission name="${prefix}_wheel_transmission" type="SimpleTransmission">
-      <type>transmission_interface/SimpleTransmission</type>
-      <joint name="${prefix}_wheel_joint">
-        <hardwareInterface>hardware_interface/EffortJointInterface</hardwareInterface>
-      </joint>
-      <actuator name="${prefix}_wheel_actuator">
-        <mechanicalReduction>1</mechanicalReduction>
-        <hardwareInterface>hardware_interface/EffortJointInterface</hardwareInterface>
-      </actuator>
-    </transmission>
     <gazebo reference="${prefix}_wheel_link">
       <mu1 value="${wheel_props['lateral_friction']}" />
@@ -77,7 +67,4 @@
       <material>Gazebo/${wheel_props['color']}</material>
     </gazebo>
-    <gazebo reference="${prefix}_wheel_joint">
-      <provideFeedback>true</provideFeedback>
-    </gazebo>
   </xacro:macro>
 </robot>
