Commit message: Update inertias for wheels, examples and GPS componnent

File: examples/dual_rplidar_s1_and_orbbec_asta/panther.urdf.xacro (robot description, xacro)
@@ -1,28 +1,49 @@
 <?xml version='1.0'?>
 <robot name="panther" xmlns:xacro="http://www.ros.org/wiki/xacro">
-  <xacro:arg name="panther_common_props_path" default="$(find panther_description)/config/panther_common.yaml" />
-  <xacro:arg name="wheel_props_path" default="$(find panther_description)/config/WH01.yaml" />
+  <xacro:arg name="use_sim" default="false" />
   <xacro:arg name="use_gpu" default="false" />
-  <!-- IMPORT YAML CONFIGS -->
-  <xacro:property name="panther_common_props_file" value="$(arg panther_common_props_path)"  />
-  <xacro:property name="panther_common_props" value="${load_yaml(panther_common_props_file)}" />
-  <xacro:property name="wheel_props_file" value="$(arg wheel_props_path)"  />
-  <xacro:property name="wheel_props" value="${load_yaml(wheel_props_file)}" />
-  <!-- INCLUDE ROBOT PARTS DEFINITIONS -->
-  <xacro:include filename="$(find panther_description)/urdf/materials.urdf.xacro" />
-  <xacro:include filename="$(find panther_description)/urdf/body.urdf.xacro" ns="body" />
-  <xacro:include filename="$(find panther_description)/urdf/wheel.urdf.xacro" ns="wheel" />
-  <xacro:include filename="$(find panther_description)/urdf/gazebo_plugins.gazebo.xacro" ns="gazebo" />
-  <!-- BODY DECLARATION -->
-  <xacro:body.body props="${panther_common_props['body']}" wheel_props="${wheel_props['wheels']}" />
-  <!-- WHEEL DECLARATION -->
-  <xacro:wheel.wheel wheel_props="${wheel_props['wheels']}" common_props="${panther_common_props}" prefix="front_left" />
-  <xacro:wheel.wheel wheel_props="${wheel_props['wheels']}" common_props="${panther_common_props}" prefix="front_right" />
-  <xacro:wheel.wheel wheel_props="${wheel_props['wheels']}" common_props="${panther_common_props}" prefix="rear_left" />
-  <xacro:wheel.wheel wheel_props="${wheel_props['wheels']}" common_props="${panther_common_props}" prefix="rear_right" />
-  <!-- GAZEBO PLUGINS -->
-  <xacro:gazebo.wheel_driver wheel_props="${wheel_props}" common_props="${panther_common_props}" />
-  <xacro:gazebo.rplidar_s1 xyz="0.185 0 0.17" rpy="0 0 0" use_gpu="$(arg use_gpu)" prefix="front" topic="laser/front/scan" />
-  <xacro:gazebo.rplidar_s1 xyz="-0.185 0 0.17" rpy="0 0 ${pi/2}" use_gpu="$(arg use_gpu)" prefix="rear" topic="laser/rear/scan" />
-  <xacro:gazebo.orbbec_astra xyz="0.36 0 0.025" rpy="0 0 0" />
+  <xacro:arg name="dual_bat" default="false" />
+  <xacro:arg name="imu_pos_x" default="0.169" />
+  <xacro:arg name="imu_pos_y" default="0.025" />
+  <xacro:arg name="imu_pos_z" default="0.092" />
+  <xacro:arg name="imu_rot_r" default="0.0" />
+  <xacro:arg name="imu_rot_p" default="0.0" />
+  <xacro:arg name="imu_rot_y" default="-1.57" />
+  <xacro:arg name="wheel_config_path" default="$(find panther_description)/config/WH01.yaml" />
+  <xacro:arg name="simulation_engine" default="gazebo-classic" />
+  <xacro:include filename="$(find panther_description)/urdf/panther_macro.urdf.xacro" ns="husarion" />
+  <xacro:husarion.panther_robot
+    use_sim="$(arg use_sim)"
+    dual_bat="$(arg dual_bat)"
+    imu_pos_x="$(arg imu_pos_x)"
+    imu_pos_y="$(arg imu_pos_y)"
+    imu_pos_z="$(arg imu_pos_z)"
+    imu_rot_r="$(arg imu_rot_r)"
+    imu_rot_p="$(arg imu_rot_p)"
+    imu_rot_y="$(arg imu_rot_y)"
+    wheel_config_path="$(arg wheel_config_path)"
+    simulation_engine="$(arg simulation_engine)" />
+  <xacro:include filename="$(find ros_components_description)/urdf/rplidar_s1.gazebo.xacro" ns="lidar" />
+  <xacro:lidar.rplidar_s1
+    parent_link="cover_link"
+    xyz="0.185 0.0 0.0"
+    rpy="0.0 0.0 0.0"
+    topic="front/scan"
+    tf_prefix="front"
+    use_gpu="$(arg use_gpu)"
+    simulation_engine="$(arg simulation_engine)" />
+  <xacro:lidar.rplidar_s1
+      parent_link="cover_link"
+      xyz="-0.185 0.0 0.0"
+      rpy="0.0 0.0 ${pi}"
+      topic="rear/scan"
+      tf_prefix="rear"
+      use_gpu="$(arg use_gpu)"
+      simulation_engine="$(arg simulation_engine)" />
+  <xacro:include filename="$(find ros_components_description)/urdf/orbbec_astra.gazebo.xacro" ns="camera" />
+  <xacro:camera.orbbec_astra
+    parent_link="front_light_link"
+    xyz="-0.01 0.0 -0.01"
+    rpy="${pi} 0.0 0.0"
+    simulation_engine="$(arg simulation_engine)" />
 </robot>

File: examples/ouster_os1_32/panther.urdf.xacro (robot description, xacro)
@@ -1,26 +1,33 @@
 <?xml version='1.0'?>
 <robot name="panther" xmlns:xacro="http://www.ros.org/wiki/xacro">
-  <xacro:arg name="panther_common_props_path" default="$(find panther_description)/config/panther_common.yaml" />
-  <xacro:arg name="wheel_props_path" default="$(find panther_description)/config/WH01.yaml" />
+  <xacro:arg name="use_sim" default="false" />
   <xacro:arg name="use_gpu" default="false" />
-  <!-- IMPORT YAML CONFIGS -->
-  <xacro:property name="panther_common_props_file" value="$(arg panther_common_props_path)"  />
-  <xacro:property name="panther_common_props" value="${load_yaml(panther_common_props_file)}" />
-  <xacro:property name="wheel_props_file" value="$(arg wheel_props_path)"  />
-  <xacro:property name="wheel_props" value="${load_yaml(wheel_props_file)}" />
-  <!-- INCLUDE ROBOT PARTS DEFINITIONS -->
-  <xacro:include filename="$(find panther_description)/urdf/materials.urdf.xacro" />
-  <xacro:include filename="$(find panther_description)/urdf/body.urdf.xacro" ns="body" />
-  <xacro:include filename="$(find panther_description)/urdf/wheel.urdf.xacro" ns="wheel" />
-  <xacro:include filename="$(find panther_description)/urdf/gazebo_plugins.gazebo.xacro" ns="gazebo" />
-  <!-- BODY DECLARATION -->
-  <xacro:body.body props="${panther_common_props['body']}" wheel_props="${wheel_props['wheels']}" />
-  <!-- WHEEL DECLARATION -->
-  <xacro:wheel.wheel wheel_props="${wheel_props['wheels']}" common_props="${panther_common_props}" prefix="front_left" />
-  <xacro:wheel.wheel wheel_props="${wheel_props['wheels']}" common_props="${panther_common_props}" prefix="front_right" />
-  <xacro:wheel.wheel wheel_props="${wheel_props['wheels']}" common_props="${panther_common_props}" prefix="rear_left" />
-  <xacro:wheel.wheel wheel_props="${wheel_props['wheels']}" common_props="${panther_common_props}" prefix="rear_right" />
-  <!-- GAZEBO PLUGINS -->
-  <xacro:gazebo.wheel_driver wheel_props="${wheel_props}" common_props="${panther_common_props}" />
-  <xacro:gazebo.ouster_os1_32 xyz="0.185 0 0.17" rpy="0 0 0" use_gpu="$(arg use_gpu)" />
+  <xacro:arg name="dual_bat" default="false" />
+  <xacro:arg name="imu_pos_x" default="0.169" />
+  <xacro:arg name="imu_pos_y" default="0.025" />
+  <xacro:arg name="imu_pos_z" default="0.092" />
+  <xacro:arg name="imu_rot_r" default="0.0" />
+  <xacro:arg name="imu_rot_p" default="0.0" />
+  <xacro:arg name="imu_rot_y" default="-1.57" />
+  <xacro:arg name="wheel_config_path" default="$(find panther_description)/config/WH01.yaml" />
+  <xacro:arg name="simulation_engine" default="gazebo-classic" />
+  <xacro:include filename="$(find panther_description)/urdf/panther_macro.urdf.xacro" ns="husarion" />
+  <xacro:husarion.panther_robot
+    use_sim="$(arg use_sim)"
+    dual_bat="$(arg dual_bat)"
+    imu_pos_x="$(arg imu_pos_x)"
+    imu_pos_y="$(arg imu_pos_y)"
+    imu_pos_z="$(arg imu_pos_z)"
+    imu_rot_r="$(arg imu_rot_r)"
+    imu_rot_p="$(arg imu_rot_p)"
+    imu_rot_y="$(arg imu_rot_y)"
+    wheel_config_path="$(arg wheel_config_path)"
+    simulation_engine="$(arg simulation_engine)" />
+  <xacro:include filename="$(find ros_components_description)/urdf/ouster_os1_32.gazebo.xacro" ns="lidar" />
+  <xacro:lidar.ouster_os1_32
+    parent_link="cover_link"
+    xyz="0.185 0.0 0.0"
+    rpy="0.0 0.0 0.0"
+    use_gpu="$(arg use_gpu)"
+    simulation_engine="$(arg simulation_engine)" />
 </robot>

File: examples/rpliar_s1_and_gps/panther.urdf.xacro (robot description, xacro)
@@ -24,3 +24,15 @@
     wheel_config_path="$(arg wheel_config_path)"
     simulation_engine="$(arg simulation_engine)" />
+  <xacro:include filename="$(find ros_components_description)/urdf/rplidar_s1.gazebo.xacro" ns="lidar" />
+  <xacro:lidar.rplidar_s1
+    parent_link="cover_link"
+    xyz="0.185 0.0 0.0"
+    rpy="0.0 0.0 0.0"
+    use_gpu="$(arg use_gpu)"
+    simulation_engine="$(arg simulation_engine)" />
+  <xacro:include filename="$(find panther_description)/urdf/components/external_antenna.urdf.xacro" ns="antenna" />
+  <xacro:antenna.external_antenna
+      parent_link="cover_link"
+      xyz="-0.1 -0.2475 0.0"
+      rpy="0.0 0.0 ${pi/2}" />
 </robot>

File: urdf/body.urdf.xacro (robot description, xacro)
@@ -26,5 +26,5 @@
       </collision>
       <inertial>
-        <origin xyz="0.0 0.0 0.0" rpy="0.0 0.0 0.0"/>
+        <origin xyz="-0.008 0.01 0.029" rpy="0.0 0.0 0.0"/>
         <mass value="43.0" />
         <inertia ixx="2.630036" ixy="-0.023480" ixz="0.052320"

File: urdf/components/external_antenna.urdf.xacro (robot description, xacro)
@@ -4,6 +4,6 @@
                params="parent_link xyz rpy
                        tf_prefix:=None
+                       frame_id:=gps
                        topic:=gps
-                       frame_id:=gps
                        initial_latitude:=53.1978
                        initial_longitude:=18.3735
@@ -27,5 +27,4 @@
         </geometry>
         <origin xyz="0.0 0.0 0.0" rpy="0.0 0.0 0.0"/>
-        <material name="DarkGrey"/>
       </visual>
       <collision>
@@ -36,10 +35,11 @@
       </collision>
       <inertial>
-          <mass value="0.105" />
-          <inertia ixx="1" ixy="0" ixz="0" iyy="1" iyz="0" izz="1" />
+        <mass value="0.59" />
+        <inertia ixx="0.003964" ixy="0.0" ixz="0.0" iyy="0.0003964" iyz="0.0" izz="0.0004177" />
+        <origin xyz="0.045 0.0 0.0058" rpy="0.0 0.0 0.0"/>
       </inertial>
     </link>
     <joint name="${tf_prefix_ext}external_antenna_link_to_${tf_prefix_ext}${frame_id}_joint" type="fixed">
-      <origin xyz="0.045 0.0 0.004" rpy="0.0 0.0 0.0" />
+      <origin xyz="0.045 0.0 0.0058" rpy="0.0 0.0 0.0" />
       <parent link="${tf_prefix_ext}external_antenna_link" />
       <child link="${tf_prefix_ext}${frame_id}" />
