Commit message: Update urdf/wheel.urdf.xacro
Co-authored-by: Maciej Stępień <maciek1284@outlook.com>

File: urdf/wheel.urdf.xacro (robot description, xacro)
@@ -28,8 +28,6 @@
       <origin xyz="${x} ${y} 0.0" rpy="0.0 0.0 0.0" />
       <axis xyz="0.0 1.0 0.0" />
-      <limit effort="34.5"
-             velocity="2.0" />
-      <dynamics damping="0.01"
-                friction="0.01"/>
+      <limit effort="34.5" velocity="2.0" />
+      <dynamics damping="0.01" friction="0.01" />
     </joint>
     <link name="${prefix}_wheel_link">

Commit message: Fix ros1 branch differences (#8)
* Fix ros1 branch differences

* Replace tabs with spaces

* Update urdf/wheel.urdf.xacro

Co-authored-by: Dawid Kmak <73443304+KmakD@users.noreply.github.com>

Co-authored-by: Dawid Kmak <73443304+KmakD@users.noreply.github.com>

File: urdf/wheel.urdf.xacro (robot description, xacro)
@@ -23,18 +23,16 @@
       <xacro:property name="inertia_y_offset" value="${-wheel_config['inertia_y_offset']}" />
     </xacro:if>
-    <joint name="${prefix}_joint" type="continuous">
+    <joint name="${prefix}_wheel_joint" type="continuous">
       <parent link="body_link" />
       <child link="${prefix}_wheel_link" />
       <origin xyz="${x} ${y} 0.0" rpy="0.0 0.0 0.0" />
       <axis xyz="0.0 1.0 0.0" />
-      <limit effort="34.5"
-             velocity="2.0" />
-      <dynamics damping="0.01"
-                friction="0.01"/>
+      <limit effort="34.5" velocity="2.0" />
+      <dynamics damping="0.01" friction="0.01" />
     </joint>
     <link name="${prefix}_wheel_link">
        <visual>
         <geometry>
-            <mesh filename="file://$(find ${wheel_config['mesh_package']})/${wheel_config['folder_path']}/${prefix}_wheel.dae" />
+          <mesh filename="file://$(find ${wheel_config['mesh_package']})/${wheel_config['folder_path']}/${prefix}_wheel.dae" />
         </geometry>
         <origin xyz="0.0 0.0 0.0" rpy="0.0 0.0 0.0" />
@@ -42,5 +40,5 @@
       <collision>
         <geometry>
-            <mesh filename="file://$(find ${wheel_config['mesh_package']})/${wheel_config['folder_path']}/collision.stl" />
+          <mesh filename="file://$(find ${wheel_config['mesh_package']})/${wheel_config['folder_path']}/collision.stl" />
         </geometry>
         <origin xyz="0.0 0.0 0.0" rpy="0.0 0.0 0.0" />
@@ -57,4 +55,11 @@
       </inertial>
     </link>
+    <gazebo reference="${prefix}_wheel_link">
+      <mu1 value="0.85" />
+      <mu2 value="0.85" />
+      <kp value="100000000.0" />
+      <kd value="5.0" />
+      <fdir1 value="1.0 0.0 0.0" />
+    </gazebo>
   </xacro:macro>
 </robot>
