Commit message: WH01 full model

File: urdf/body.urdf.xacro (robot description, xacro)
@@ -2,5 +2,8 @@
 <robot xmlns:xacro="http://www.ros.org/wiki/xacro">
   <!-- body defining macro -->
-  <xacro:macro name="body" params="wheel_diameter">
+  <xacro:macro name="body" params="
+    wheel_diameter simulation_engine
+    imu_pos_x imu_pos_y imu_pos_z
+    imu_rot_r imu_rot_p imu_rot_y" >
     <link name="base_link"></link>
     <link name="body_link">
@@ -25,5 +28,4 @@
     </link>
     <link name="imu_link"></link>
-    <link name="gps_link"></link>
     <link name="front_light_link"></link>
     <link name="rear_light_link"></link>
@@ -35,71 +37,43 @@
     </joint>
     <joint name="body_link_to_imu_link_joint" type="fixed">
-      <origin xyz="0.169 0.025 0.092" rpy="0.0 0.0 0.0" />
+      <origin xyz="${imu_pos_x} ${imu_pos_y} ${imu_pos_z}"
+              rpy="${imu_rot_r} ${imu_rot_p} ${imu_rot_y}" />
       <parent link="body_link" />
       <child link="imu_link" />
     </joint>
-    <joint name="body_link_to_gps_link_joint" type="fixed">
-      <origin xyz="0.0 0.0 0.0" rpy="0.0 0.0 0.0" />
-      <parent link="body_link" />
-      <child link="gps_link" />
-    </joint>
     <joint name="body_link_front_light_link_joint" type="fixed">
-      <origin xyz="0.0 0.0 0.0" rpy="0.0 0.0 0.0" />
+      <origin xyz="0.362 0.0 0.0" rpy="0.0 0.0 0.0" />
       <parent link="body_link" />
       <child link="front_light_link" />
     </joint>
     <joint name="body_link_to_rear_light_link_joint" type="fixed">
-      <origin xyz="0.0 0.0 0.0" rpy="0.0 0.0 0.0" />
+      <origin xyz="-0.362 0.0 0.0" rpy="0.0 0.0 ${pi}" />
       <parent link="body_link" />
       <child link="rear_light_link" />
     </joint>
     <joint name="body_link_to_cover_link_joint" type="fixed">
-      <origin xyz="0.0 0.0 0.17" rpy="0.0 0.0 0.0" />
+      <origin xyz="0.0 0.0 0.1715" rpy="0.0 0.0 0.0" />
       <parent link="body_link" />
       <child link="cover_link" />
     </joint>
-    <!-- publish joint states -->
-    <gazebo>
-      <plugin name="joint_states" filename="libgazebo_ros_joint_state_publisher.so">
-        <joint_name>front_left_wheel_joint</joint_name>
-        <joint_name>front_right_wheel_joint</joint_name>
-        <joint_name>rear_left_wheel_joint</joint_name>
-        <joint_name>rear_right_wheel_joint</joint_name>
-      </plugin>
-    </gazebo>
-    <!-- based on PhidgetSpatial datasheet -->
-    <xacro:property name="imu_acc_noise"  value="${280.0*1e-6*9.81}" />
-    <xacro:property name="imu_acc_drift"  value="${40.6*1e-6*9.81}" />
-    <xacro:property name="imu_gyro_noise" value="${0.095*(pi/180.0)}" />
-    <xacro:property name="imu_gyro_drift" value="${0.0042*(pi/180.0)}" />
-    <gazebo>
-      <plugin name="imu_controller" filename="libhector_gazebo_ros_imu.so">
-        <robotNamespace>/</robotNamespace>
-        <updateRate>100.0</updateRate>
-        <bodyName>imu_link</bodyName>
-        <topicName>imu</topicName>
-        <accelDrift>${imu_acc_drift} ${imu_acc_drift} ${imu_acc_drift}</accelDrift>
-        <accelGaussianNoise>${imu_acc_noise} ${imu_acc_noise} ${imu_acc_noise}</accelGaussianNoise>
-        <rateDrift>${imu_gyro_drift} ${imu_gyro_drift} ${imu_gyro_drift}</rateDrift>
-        <rateGaussianNoise>${imu_gyro_noise} ${imu_gyro_noise} ${imu_gyro_noise}</rateGaussianNoise>
-      </plugin>
-    </gazebo>
-    <!-- based on Teltonika RUTX11 datasheet and measuremets-->
-    <gazebo>
-      <plugin name="gps_controller" filename="libhector_gazebo_ros_gps.so">
-        <updateRate>40</updateRate>
-        <robotNamespace>/</robotNamespace>
-        <bodyName>gps_link</bodyName>
-        <frameId>gps_link</frameId>
-        <topicName>/global_position/fix</topicName>
-        <velocityTopicName>/global_position/vel</velocityTopicName>
-        <referenceLatitude>53.1978</referenceLatitude>
-        <referenceLongitude>18.3735</referenceLongitude>
-        <referenceHeading>0</referenceHeading>
-        <referenceAltitude>0</referenceAltitude>
-        <drift>0.0001 0.0001 0.0001</drift>
-        <gaussianNoise>3.0 3.0 3.0</gaussianNoise>
-      </plugin>
-    </gazebo>
+    <xacro:if value="${simulation_engine == 'gazebo-classic'}">
+      <!-- based on PhidgetSpatial datasheet -->
+      <xacro:property name="imu_acc_noise"  value="${280.0*1e-6*9.81}" />
+      <xacro:property name="imu_acc_drift"  value="${40.6*1e-6*9.81}" />
+      <xacro:property name="imu_gyro_noise" value="${0.095*(pi/180.0)}" />
+      <xacro:property name="imu_gyro_drift" value="${0.0042*(pi/180.0)}" />
+      <gazebo>
+        <plugin name="imu_controller" filename="libhector_gazebo_ros_imu.so">
+          <robotNamespace>/</robotNamespace>
+          <updateRate>100.0</updateRate>
+          <bodyName>imu_link</bodyName>
+          <topicName>imu</topicName>
+          <accelDrift>${imu_acc_drift} ${imu_acc_drift} ${imu_acc_drift}</accelDrift>
+          <accelGaussianNoise>${imu_acc_noise} ${imu_acc_noise} ${imu_acc_noise}</accelGaussianNoise>
+          <rateDrift>${imu_gyro_drift} ${imu_gyro_drift} ${imu_gyro_drift}</rateDrift>
+          <rateGaussianNoise>${imu_gyro_noise} ${imu_gyro_noise} ${imu_gyro_noise}</rateGaussianNoise>
+        </plugin>
+      </gazebo>
+  </xacro:if>
   </xacro:macro>
 </robot>

File: urdf/panther.urdf.xacro (robot description, xacro)
@@ -3,14 +3,28 @@
   <xacro:arg name="use_sim" default="false" />
   <xacro:arg name="use_gpu" default="false" />
-  <xacro:arg name="has_gps" default="false" />
-  <xacro:arg name="wheel_props_path" default="$(find panther_description)/urdf/config/WH01.yaml" />
+  <xacro:arg name="dual_bat" default="false" />
+  <xacro:arg name="imu_pos_x" default="0.169" />
+  <xacro:arg name="imu_pos_y" default="0.025" />
+  <xacro:arg name="imu_pos_z" default="0.092" />
+  <xacro:arg name="imu_rot_r" default="0.0" />
+  <xacro:arg name="imu_rot_p" default="0.0" />
+  <xacro:arg name="imu_rot_y" default="-1.57" />
+  <xacro:arg name="wheel_props_path" default="$(find panther_description)/config/WH01.yaml" />
+  <xacro:arg name="simulation_engine" default="gazebo-classic" />
   <xacro:include filename="$(find panther_description)/urdf/panther_macro.urdf.xacro" ns="husarion" />
   <xacro:husarion.panther_robot
     use_sim="$(arg use_sim)"
     use_gpu="$(arg use_gpu)"
-    has_gps="$(arg has_gps)"
+    dual_bat="$(arg dual_bat)"
+    imu_pos_x="$(arg imu_pos_x)"
+    imu_pos_y="$(arg imu_pos_y)"
+    imu_pos_z="$(arg imu_pos_z)"
+    imu_rot_r="$(arg imu_rot_r)"
+    imu_rot_p="$(arg imu_rot_p)"
+    imu_rot_y="$(arg imu_rot_y)"
     wheel_props_path="$(arg wheel_props_path)"
+    simulation_engine="$(arg simulation_engine)"
   />
-  <xacro:include filename="$(find panther_description)/urdf/components/orbbec_astra.gazebo.xacro" ns="lidar" />
-  <xacro:lidar.orbbec_astra parent_link="cover_link" xyz="0.185 0.0 0.0" rpy="0.0 0.0 0.0" use_gpu="$(arg use_gpu)" />
+  <!-- <xacro:include filename="$(find components_description)/urdf/orbbec_astra.gazebo.xacro" ns="lidar" /> -->
+  <!-- <xacro:lidar.orbbec_astra parent_link="cover_link" xyz="0.185 0.0 0.0" rpy="0.0 0.0 0.0" use_gpu="$(arg use_gpu)" /> -->
 </robot>

File: urdf/panther_macro.urdf.xacro (robot description, xacro)
@@ -3,7 +3,14 @@
   <xacro:macro name="panther_robot"
                params="use_sim:=false
-                       use_gpu:=true
-                       has_gps:=false
-                       wheel_props_path:=None">
+                       use_gpu:=false
+                       dual_bat:=false
+                       imu_pos_x:=0.169
+                       imu_pos_y:=0.025
+                       imu_pos_z:=0.092
+                       imu_rot_r:=0.0
+                       imu_rot_p:=0.0
+                       imu_rot_y:=-1.57
+                       wheel_props_path:=None
+                       simulation_engine:='gazebo-classic'">
     <xacro:if value="${wheel_props_path == 'None'}">
       <xacro:property name="wheel_props_file" value="$(find panther_description)/config/WH01.yaml"  />
@@ -17,5 +24,13 @@
     <xacro:include filename="$(find panther_description)/urdf/wheel.urdf.xacro" ns="wheel" />
     <!-- BODY DECLARATION -->
-    <xacro:body.body wheel_diameter="${wheel_props['wheels']['diameter']}" />
+    <xacro:body.body
+      wheel_diameter="${wheel_props['wheels']['diameter']}"
+      imu_pos_x="${imu_pos_x}"
+      imu_pos_y="${imu_pos_y}"
+      imu_pos_z="${imu_pos_z}"
+      imu_rot_r="${imu_rot_r}"
+      imu_rot_p="${imu_rot_p}"
+      imu_rot_y="${imu_rot_y}"
+      simulation_engine="${simulation_engine}" />
     <!-- WHEEL DECLARATION -->
     <xacro:wheel.wheel wheel_props="${wheel_props['wheels']}" prefix="front_left" />
@@ -23,46 +38,56 @@
     <xacro:wheel.wheel wheel_props="${wheel_props['wheels']}" prefix="rear_left" />
     <xacro:wheel.wheel wheel_props="${wheel_props['wheels']}" prefix="rear_right" />
-    <xacro:if value="${wheel_props['wheels']['kinematics'] == 'classic'}">
+    <xacro:if value="${simulation_engine == 'gazebo-classic'}">
       <gazebo>
-        <plugin name='skid_steer_drive' filename='libgazebo_ros_diff_drive.so'>
-          <ros>
-          </ros>
-          <update_rate>10</update_rate>
-          <num_wheel_pairs>2</num_wheel_pairs>
-          <left_joint>front_left_wheel_joint</left_joint>
-          <right_joint>front_right_wheel_joint</right_joint>
-          <left_joint>rear_left_wheel_joint</left_joint>
-          <right_joint>rear_right_wheel_joint</right_joint>
-          <wheel_separation>${wheel_props['wheels']['wheel_separation']}</wheel_separation>
-          <wheel_separation>${wheel_props['wheels']['wheel_separation']}</wheel_separation>
-          <wheel_diameter>${wheel_props['wheels']['diameter']}</wheel_diameter>
-          <wheel_diameter>${wheel_props['wheels']['diameter']}</wheel_diameter>
-          <max_wheel_torque>34.5</max_wheel_torque>
-          <max_wheel_acceleration>2.0</max_wheel_acceleration>
-          <publish_odom>true</publish_odom>
-          <publish_odom_tf>true</publish_odom_tf>
-          <publish_wheel_tf>true</publish_wheel_tf>
-          <odometry_frame>odom</odometry_frame>
-          <robot_base_frame>base_link</robot_base_frame>
+        <plugin name="joint_states" filename="libgazebo_ros_joint_state_publisher.so">
+          <joint_name>front_left_wheel_joint</joint_name>
+          <joint_name>front_right_wheel_joint</joint_name>
+          <joint_name>rear_left_wheel_joint</joint_name>
+          <joint_name>rear_right_wheel_joint</joint_name>
         </plugin>
       </gazebo>
-    </xacro:if>
-    <xacro:if value="${wheel_props['wheels']['kinematics'] == 'mecanum'}">
-      <gazebo>
-        <plugin name="object_controller" filename="libgazebo_ros_planar_move.so">
-          <ros>
-          </ros>
-          <update_rate>10</update_rate>
-          <publish_rate>10</publish_rate>
-          <publish_odom>true</publish_odom>
-          <publish_odom_tf>true</publish_odom_tf>
-          <odometry_frame>odom</odometry_frame>
-          <robot_base_frame>base_link</robot_base_frame>
-          <covariance_x>0.0001</covariance_x>
-          <covariance_y>0.0001</covariance_y>
-          <covariance_yaw>0.01</covariance_yaw>
-        </plugin>
-      </gazebo>
-    </xacro:if>
+      <xacro:if value="${wheel_props['wheels']['kinematics'] == 'classic'}">
+        <gazebo>
+          <plugin name='skid_steer_drive' filename='libgazebo_ros_diff_drive.so'>
+            <ros>
+            </ros>
+            <update_rate>10</update_rate>
+            <num_wheel_pairs>2</num_wheel_pairs>
+            <left_joint>front_left_wheel_joint</left_joint>
+            <right_joint>front_right_wheel_joint</right_joint>
+            <left_joint>rear_left_wheel_joint</left_joint>
+            <right_joint>rear_right_wheel_joint</right_joint>
+            <wheel_separation>${wheel_props['wheels']['wheel_separation']}</wheel_separation>
+            <wheel_separation>${wheel_props['wheels']['wheel_separation']}</wheel_separation>
+            <wheel_diameter>${wheel_props['wheels']['diameter']}</wheel_diameter>
+            <wheel_diameter>${wheel_props['wheels']['diameter']}</wheel_diameter>
+            <max_wheel_torque>34.5</max_wheel_torque>
+            <max_wheel_acceleration>2.0</max_wheel_acceleration>
+            <publish_odom>true</publish_odom>
+            <publish_odom_tf>true</publish_odom_tf>
+            <publish_wheel_tf>true</publish_wheel_tf>
+            <odometry_frame>odom</odometry_frame>
+            <robot_base_frame>base_link</robot_base_frame>
+          </plugin>
+        </gazebo>
+      </xacro:if>
+      <xacro:if value="${wheel_props['wheels']['kinematics'] == 'mecanum'}">
+        <gazebo>
+          <plugin name="object_controller" filename="libgazebo_ros_planar_move.so">
+            <ros>
+            </ros>
+            <update_rate>10</update_rate>
+            <publish_rate>10</publish_rate>
+            <publish_odom>true</publish_odom>
+            <publish_odom_tf>true</publish_odom_tf>
+            <odometry_frame>odom</odometry_frame>
+            <robot_base_frame>base_link</robot_base_frame>
+            <covariance_x>0.0001</covariance_x>
+            <covariance_y>0.0001</covariance_y>
+            <covariance_yaw>0.01</covariance_yaw>
+          </plugin>
+        </gazebo>
+      </xacro:if>
+  </xacro:if>
   </xacro:macro>
 </robot>

File: urdf/wheel.urdf.xacro (robot description, xacro)
@@ -5,24 +5,51 @@
     <xacro:property name="wheel_separation_x" value="0.44" />
     <xacro:property name="rpy" value="0 0 0" />
-    <xacro:property name="mesh_folder" value="${wheel_props['mesh_folder']}" />
     <xacro:if value="${prefix == 'front_left'}">
-      <xacro:property name="x" value="${wheel_separation_x/2}" />
-      <xacro:property name="y" value="${wheel_props['wheel_separation']/2}" />
-      <xacro:property name="mesh" value="file://$(find panther_description)/meshes/${mesh_folder}/wheel_a.dae" />
+      <xacro:property name="x" value="${wheel_separation_x/2.0}" />
+      <xacro:property name="y" value="${wheel_props['wheel_separation']/2.0}" />
+      <xacro:if value="${wheel_props['kinematics'] == 'classic'}">
+        <xacro:property name="mesh"
+          value="file://$(find ${wheel_props['mesh_package']})/${wheel_props['folder_path']}/wheel_a.dae" />
+      </xacro:if>
+      <xacro:if value="${wheel_props['kinematics'] == 'mecanum'}">
+        <xacro:property name="mesh"
+          value="file://$(find ${wheel_props['mesh_package']})/${wheel_props['folder_path']}/wheel_a.dae" />
+      </xacro:if>
     </xacro:if>
     <xacro:if value="${prefix == 'front_right'}">
-      <xacro:property name="x" value="${wheel_separation_x/2}" />
-      <xacro:property name="y" value="-${wheel_props['wheel_separation']/2}" />
-      <xacro:property name="mesh" value="file://$(find panther_description)/meshes/${mesh_folder}/wheel_b.dae" />
+      <xacro:property name="x" value="${wheel_separation_x/2.0}" />
+      <xacro:property name="y" value="-${wheel_props['wheel_separation']/2.0}" />
+      <xacro:if value="${wheel_props['kinematics'] == 'classic'}">
+        <xacro:property name="mesh"
+          value="file://$(find ${wheel_props['mesh_package']})/${wheel_props['folder_path']}/wheel_b.dae" />
+      </xacro:if>
+      <xacro:if value="${wheel_props['kinematics'] == 'mecanum'}">
+        <xacro:property name="mesh"
+          value="file://$(find ${wheel_props['mesh_package']})/${wheel_props['folder_path']}/wheel_b.dae" />
+      </xacro:if>
     </xacro:if>
     <xacro:if value="${prefix == 'rear_left'}">
-      <xacro:property name="x" value="-${wheel_separation_x/2}" />
-      <xacro:property name="y" value="${wheel_props['wheel_separation']/2}" />
-      <xacro:property name="mesh" value="file://$(find panther_description)/meshes/${mesh_folder}/wheel_a.dae" />
+      <xacro:property name="x" value="-${wheel_separation_x/2.0}" />
+      <xacro:property name="y" value="${wheel_props['wheel_separation']/2.0}" />
+      <xacro:if value="${wheel_props['kinematics'] == 'classic'}">
+        <xacro:property name="mesh"
+          value="file://$(find ${wheel_props['mesh_package']})/${wheel_props['folder_path']}/wheel_a.dae" />
+      </xacro:if>
+      <xacro:if value="${wheel_props['kinematics'] == 'mecanum'}">
+        <xacro:property name="mesh"
+          value="file://$(find ${wheel_props['mesh_package']})/${wheel_props['folder_path']}/wheel_c.dae" />
+      </xacro:if>
     </xacro:if>
     <xacro:if value="${prefix == 'rear_right'}">
-      <xacro:property name="x" value="-${wheel_separation_x/2}" />
-      <xacro:property name="y" value="-${wheel_props['wheel_separation']/2}" />
-      <xacro:property name="mesh" value="file://$(find panther_description)/meshes/${mesh_folder}/wheel_b.dae" />
+      <xacro:property name="x" value="-${wheel_separation_x/2.0}" />
+      <xacro:property name="y" value="-${wheel_props['wheel_separation']/2.0}" />
+      <xacro:if value="${wheel_props['kinematics'] == 'classic'}">
+        <xacro:property name="mesh"
+          value="file://$(find ${wheel_props['mesh_package']})/${wheel_props['folder_path']}/wheel_b.dae" />
+      </xacro:if>
+      <xacro:if value="${wheel_props['kinematics'] == 'mecanum'}">
+        <xacro:property name="mesh"
+          value="file://$(find ${wheel_props['mesh_package']})/${wheel_props['folder_path']}/wheel_d.dae" />
+      </xacro:if>
     </xacro:if>
     <link name="${prefix}_wheel_link">
@@ -35,5 +62,5 @@
       <collision>
         <geometry>
-            <mesh filename="file://$(find panther_description)/meshes/${mesh_folder}/collision.stl" scale="1.0 1.0 1.0" />
+            <mesh filename="file://$(find ${wheel_props['mesh_package']})/${wheel_props['folder_path']}/collision.stl" scale="1.0 1.0 1.0" />
         </geometry>
         <origin xyz="0.0 0.0 0.0" rpy="0.0 0.0 0.0" />
