Commit message: Update README, package.xml and setup simulation

File: urdf/body.urdf.xacro (robot description, xacro)
@@ -21,8 +21,9 @@
       </collision>
       <inertial>
-          <mass value="43.0" />
-          <inertia ixx="2.630036" ixy="-0.023480" ixz="0.052320"
-                                  iyy="2.463509"  iyz="0.009337"
-                                                  izz="4.611945" />
+        <origin xyz="0.0 0.0 0.0" rpy="0.0 0.0 0.0"/>
+        <mass value="43.0" />
+        <inertia ixx="2.630036" ixy="-0.023480" ixz="0.052320"
+                                iyy="2.463509"  iyz="0.009337"
+                                                izz="4.611945" />
       </inertial>
     </link>

File: urdf/panther.urdf.xacro (robot description, xacro)
@@ -24,7 +24,11 @@
     imu_rot_y="$(arg imu_rot_y)"
     wheel_props_path="$(arg wheel_props_path)"
-    simulation_engine="$(arg simulation_engine)"
-  />
-  <!-- <xacro:include filename="$(find components_description)/urdf/orbbec_astra.gazebo.xacro" ns="lidar" /> -->
-  <!-- <xacro:lidar.orbbec_astra parent_link="cover_link" xyz="0.185 0.0 0.0" rpy="0.0 0.0 0.0" use_gpu="$(arg use_gpu)" /> -->
+    simulation_engine="$(arg simulation_engine)" />
+  <xacro:include filename="$(find ros_components_description)/urdf/rplidar_s1.gazebo.xacro" ns="lidar" />
+  <xacro:lidar.rplidar_s1
+    parent_link="cover_link"
+    xyz="0.185 0.0 0.0"
+    rpy="0.0 0.0 0.0"
+    use_gpu="$(arg use_gpu)"
+    simulation_engine="$(arg simulation_engine)" />
 </robot>

File: urdf/panther_macro.urdf.xacro (robot description, xacro)
@@ -40,5 +40,5 @@
     <xacro:if value="${simulation_engine == 'gazebo-classic'}">
       <gazebo>
-        <plugin name="joint_states" filename="libgazebo_ros_joint_state_publisher.so">
+          <plugin name="joint_states" filename="libgazebo_ros_joint_state_publisher.so">
           <joint_name>front_left_wheel_joint</joint_name>
           <joint_name>front_right_wheel_joint</joint_name>
@@ -47,5 +47,5 @@
         </plugin>
       </gazebo>
-      <xacro:if value="${wheel_props['wheels']['kinematics'] == 'classic'}">
+      <xacro:if value="${wheel_props['wheels']['kinematics'] == 'differential'}">
         <gazebo>
           <plugin name='skid_steer_drive' filename='libgazebo_ros_diff_drive.so'>

File: urdf/wheel.urdf.xacro (robot description, xacro)
@@ -8,48 +8,28 @@
       <xacro:property name="x" value="${wheel_separation_x/2.0}" />
       <xacro:property name="y" value="${wheel_props['wheel_separation']/2.0}" />
-      <xacro:if value="${wheel_props['kinematics'] == 'classic'}">
-        <xacro:property name="mesh"
-          value="file://$(find ${wheel_props['mesh_package']})/${wheel_props['folder_path']}/wheel_a.dae" />
-      </xacro:if>
-      <xacro:if value="${wheel_props['kinematics'] == 'mecanum'}">
-        <xacro:property name="mesh"
-          value="file://$(find ${wheel_props['mesh_package']})/${wheel_props['folder_path']}/wheel_a.dae" />
-      </xacro:if>
+      <xacro:property name="inertia_y_offset" value="${wheel_props['inertia_y_offset']}" />
+      <xacro:property name="mesh"
+        value="file://$(find ${wheel_props['mesh_package']})/${wheel_props['folder_path']}/wheel_a.dae" />
     </xacro:if>
     <xacro:if value="${prefix == 'front_right'}">
       <xacro:property name="x" value="${wheel_separation_x/2.0}" />
       <xacro:property name="y" value="-${wheel_props['wheel_separation']/2.0}" />
-      <xacro:if value="${wheel_props['kinematics'] == 'classic'}">
-        <xacro:property name="mesh"
-          value="file://$(find ${wheel_props['mesh_package']})/${wheel_props['folder_path']}/wheel_b.dae" />
-      </xacro:if>
-      <xacro:if value="${wheel_props['kinematics'] == 'mecanum'}">
-        <xacro:property name="mesh"
-          value="file://$(find ${wheel_props['mesh_package']})/${wheel_props['folder_path']}/wheel_b.dae" />
-      </xacro:if>
+      <xacro:property name="inertia_y_offset" value="${-wheel_props['inertia_y_offset']}" />
+      <xacro:property name="mesh"
+        value="file://$(find ${wheel_props['mesh_package']})/${wheel_props['folder_path']}/wheel_b.dae" />
     </xacro:if>
     <xacro:if value="${prefix == 'rear_left'}">
       <xacro:property name="x" value="-${wheel_separation_x/2.0}" />
       <xacro:property name="y" value="${wheel_props['wheel_separation']/2.0}" />
-      <xacro:if value="${wheel_props['kinematics'] == 'classic'}">
-        <xacro:property name="mesh"
-          value="file://$(find ${wheel_props['mesh_package']})/${wheel_props['folder_path']}/wheel_a.dae" />
-      </xacro:if>
-      <xacro:if value="${wheel_props['kinematics'] == 'mecanum'}">
-        <xacro:property name="mesh"
-          value="file://$(find ${wheel_props['mesh_package']})/${wheel_props['folder_path']}/wheel_c.dae" />
-      </xacro:if>
+      <xacro:property name="inertia_y_offset" value="${wheel_props['inertia_y_offset']}" />
+      <xacro:property name="mesh"
+        value="file://$(find ${wheel_props['mesh_package']})/${wheel_props['folder_path']}/wheel_c.dae" />
     </xacro:if>
     <xacro:if value="${prefix == 'rear_right'}">
       <xacro:property name="x" value="-${wheel_separation_x/2.0}" />
       <xacro:property name="y" value="-${wheel_props['wheel_separation']/2.0}" />
-      <xacro:if value="${wheel_props['kinematics'] == 'classic'}">
-        <xacro:property name="mesh"
-          value="file://$(find ${wheel_props['mesh_package']})/${wheel_props['folder_path']}/wheel_b.dae" />
-      </xacro:if>
-      <xacro:if value="${wheel_props['kinematics'] == 'mecanum'}">
-        <xacro:property name="mesh"
-          value="file://$(find ${wheel_props['mesh_package']})/${wheel_props['folder_path']}/wheel_d.dae" />
-      </xacro:if>
+      <xacro:property name="inertia_y_offset" value="${-wheel_props['inertia_y_offset']}" />
+      <xacro:property name="mesh"
+        value="file://$(find ${wheel_props['mesh_package']})/${wheel_props['folder_path']}/wheel_d.dae" />
     </xacro:if>
     <link name="${prefix}_wheel_link">
@@ -67,11 +47,12 @@
       </collision>
       <inertial>
-          <mass value="${wheel_props['mass']}" />
-          <inertia ixx="${wheel_props['inertia']['ixx']}"
-                   ixy="${wheel_props['inertia']['ixy']}"
-                   ixz="${wheel_props['inertia']['ixz']}"
-                   iyy="${wheel_props['inertia']['iyy']}"
-                   iyz="${wheel_props['inertia']['iyz']}"
-                   izz="${wheel_props['inertia']['izz']}" />
+        <origin xyz="0.0 ${inertia_y_offset} 0.0" rpy="0.0 0.0 0.0"/>
+        <mass value="${wheel_props['mass']}" />
+        <inertia ixx="${wheel_props['inertia']['ixx']}"
+                 ixy="0.0"
+                 ixz="0.0"
+                 iyy="${wheel_props['inertia']['iyy']}"
+                 iyz="0.0"
+                 izz="${wheel_props['inertia']['izz']}" />
       </inertial>
     </link>

Commit message: Update changes from review

File: urdf/body.urdf.xacro (robot description, xacro)
@@ -3,5 +3,5 @@
   <!-- body defining macro -->
   <xacro:macro name="body" params="
-    wheel_diameter simulation_engine
+    wheel_radius simulation_engine
     imu_pos_x imu_pos_y imu_pos_z
     imu_rot_r imu_rot_p imu_rot_y" >
@@ -10,5 +10,5 @@
       <visual>
         <geometry>
-          <mesh filename="file://$(find panther_description)/meshes/body.dae" scale="1.0 1.0 1.0" />
+          <mesh filename="file://$(find panther_description)/meshes/body.dae" />
         </geometry>
         <origin xyz="0.0 0.0 0.0" rpy="0.0 0.0 0.0"/>
@@ -16,5 +16,5 @@
       <collision>
         <geometry>
-          <mesh filename="file://$(find panther_description)/meshes/body_collision.stl" scale="1.0 1.0 1.0" />
+          <mesh filename="file://$(find panther_description)/meshes/body_collision.stl" />
         </geometry>
         <origin xyz="0.0 0.0 0.0" rpy="0.0 0.0 0.0"/>
@@ -33,5 +33,5 @@
     <link name="cover_link"></link>
     <joint name="base_link_to_body_link_joint" type="fixed">
-      <origin xyz="0.0 0.0 ${wheel_diameter/2.0}" rpy="0.0 0.0 0.0" />
+      <origin xyz="0.0 0.0 ${wheel_radius}" rpy="0.0 0.0 0.0" />
       <parent link="base_link" />
       <child link="body_link" />

File: urdf/components/external_antenna.urdf.xacro (robot description, xacro)
@@ -5,5 +5,6 @@
                        tf_prefix:=None
                        topic:=gps
-                       frame_id:=gps">
+                       frame_id:=gps
+                       simulation_engine:=gazebo-classic">
     <xacro:if value="${tf_prefix == 'None'}">
       <xacro:property name="tf_prefix_ext" value="" />
@@ -12,8 +13,8 @@
       <xacro:property name="tf_prefix_ext" value="${tf_prefix}_" />
     </xacro:unless>
-    <link name="${tf_prefix_ext}${frame_id}">
+    <link name="${tf_prefix_ext}external_antenna_link">
       <visual>
         <geometry>
-          <mesh filename="file://$(find panther_description)/meshes/components/external_antenna.stl" scale="0.001 0.001 0.001" />
+          <mesh filename="file://$(find panther_description)/meshes/components/external_antenna.dae" />
         </geometry>
         <origin xyz="0.0 0.0 0.0" rpy="0.0 0.0 0.0"/>
@@ -22,5 +23,5 @@
       <collision>
         <geometry>
-          <mesh filename="file://$(find panther_description)/meshes/components/external_antenna.stl" scale="0.001 0.001 0.001" />
+          <mesh filename="file://$(find panther_description)/meshes/components/external_antenna.dae" />
         </geometry>
         <origin xyz="0.0 0.0 0.0" rpy="0.0 0.0 0.0"/>
@@ -31,7 +32,13 @@
       </inertial>
     </link>
-    <joint name="${parent_link}_to_${tf_prefix_ext}${frame_id}_joint" type="fixed">
+    <joint name="${parent_link}_to_${tf_prefix_ext}external_antenna_link_joint" type="fixed">
       <origin xyz="${xyz}" rpy="${rpy}" />
       <parent link="${parent_link}" />
+      <child link="${tf_prefix_ext}external_antenna_link" />
+    </joint>
+    <link name="${tf_prefix_ext}${frame_id}"></link>
+    <joint name="${tf_prefix_ext}external_antenna_link_to_${tf_prefix_ext}${frame_id}_joint" type="fixed">
+      <origin xyz="0.0 0.0 0.0" rpy="0.0 0.0 0.0" />
+      <parent link="${tf_prefix_ext}external_antenna_link" />
       <child link="${tf_prefix_ext}${frame_id}" />
     </joint>

File: urdf/panther.urdf.xacro (robot description, xacro)
@@ -10,5 +10,5 @@
   <xacro:arg name="imu_rot_p" default="0.0" />
   <xacro:arg name="imu_rot_y" default="-1.57" />
-  <xacro:arg name="wheel_props_path" default="$(find panther_description)/config/WH01.yaml" />
+  <xacro:arg name="wheel_config_path" default="$(find panther_description)/config/WH01.yaml" />
   <xacro:arg name="simulation_engine" default="gazebo-classic" />
   <xacro:include filename="$(find panther_description)/urdf/panther_macro.urdf.xacro" ns="husarion" />
@@ -22,7 +22,7 @@
     imu_rot_p="$(arg imu_rot_p)"
     imu_rot_y="$(arg imu_rot_y)"
-    wheel_props_path="$(arg wheel_props_path)"
+    wheel_config_path="$(arg wheel_config_path)"
     simulation_engine="$(arg simulation_engine)" />
-  <xacro:include filename="$(find ros_components_description)/urdf/rplidar_s1.gazebo.xacro" ns="lidar" />
+  <!-- <xacro:include filename="$(find ros_components_description)/urdf/rplidar_s1.gazebo.xacro" ns="lidar" />
   <xacro:lidar.rplidar_s1
     parent_link="cover_link"
@@ -30,4 +30,9 @@
     rpy="0.0 0.0 0.0"
     use_gpu="$(arg use_gpu)"
-    simulation_engine="$(arg simulation_engine)" />
+    simulation_engine="$(arg simulation_engine)" /> -->
+  <xacro:include filename="$(find panther_description)/urdf/components/external_antenna.urdf.xacro" ns="antenna" />
+  <xacro:antenna.external_antenna
+    parent_link="cover_link"
+    xyz="0.0 0.0 0.0"
+    rpy="0.0 0.0 0.0" />
 </robot>

File: urdf/panther_macro.urdf.xacro (robot description, xacro)
@@ -4,19 +4,20 @@
                params="use_sim:=false
                        dual_bat:=false
-                       imu_pos_x:=0.169
-                       imu_pos_y:=0.025
-                       imu_pos_z:=0.092
-                       imu_rot_r:=0.0
-                       imu_rot_p:=0.0
-                       imu_rot_y:=-1.57
-                       wheel_props_path:=None
+                       imu_pos_x:=0.168
+                       imu_pos_y:=0.028
+                       imu_pos_z:=0.083
+                       imu_rot_r:=3.14
+                       imu_rot_p:=-1.57
+                       imu_rot_y:=0.0
+                       wheel_config_path:=None
                        simulation_engine:='gazebo-classic'">
-    <xacro:if value="${wheel_props_path == 'None'}">
-      <xacro:property name="wheel_props_file" value="$(find panther_description)/config/WH01.yaml"  />
+    <xacro:if value="${wheel_config_path == 'None'}">
+      <xacro:property name="wheel_config_file" value="$(find panther_description)/config/WH01.yaml"  />
     </xacro:if>
-    <xacro:unless value="${wheel_props_path == 'None'}">
-      <xacro:property name="wheel_props_file" value="$(arg wheel_props_path)"  />
+    <xacro:unless value="${wheel_config_path == 'None'}">
+      <xacro:property name="wheel_config_file" value="$(arg wheel_config_path)"  />
     </xacro:unless>
-    <xacro:property name="wheel_props" value="${load_yaml(wheel_props_file)}" />
+    <xacro:property name="wheel_config_ros_params" value="${load_yaml(wheel_config_file)}" />
+    <xacro:property name="wheel_config" value="${wheel_config_ros_params['/**']['ros__parameters']}" />
     <!-- INCLUDE ROBOT PARTS DEFINITIONS -->
     <xacro:include filename="$(find panther_description)/urdf/body.urdf.xacro" ns="body" />
@@ -24,5 +25,5 @@
     <!-- BODY DECLARATION -->
     <xacro:body.body
-      wheel_diameter="${wheel_props['wheels']['diameter']}"
+      wheel_radius="${wheel_config['wheel_radius']}"
       imu_pos_x="${imu_pos_x}"
       imu_pos_y="${imu_pos_y}"
@@ -32,19 +33,32 @@
       imu_rot_y="${imu_rot_y}"
       simulation_engine="${simulation_engine}" />
+    <xacro:property name="wheel_separation_x" value="0.44" />
     <!-- WHEEL DECLARATION -->
-    <xacro:wheel.wheel wheel_props="${wheel_props['wheels']}" prefix="front_left" />
-    <xacro:wheel.wheel wheel_props="${wheel_props['wheels']}" prefix="front_right" />
-    <xacro:wheel.wheel wheel_props="${wheel_props['wheels']}" prefix="rear_left" />
-    <xacro:wheel.wheel wheel_props="${wheel_props['wheels']}" prefix="rear_right" />
+    <xacro:wheel.wheel
+      wheel_config="${wheel_config}"
+      wheel_separation_x="${wheel_separation_x}"
+      prefix="fl" />
+    <xacro:wheel.wheel
+      wheel_config="${wheel_config}"
+      wheel_separation_x="${wheel_separation_x}"
+      prefix="fr" />
+    <xacro:wheel.wheel
+      wheel_config="${wheel_config}"
+      wheel_separation_x="${wheel_separation_x}"
+      prefix="rl" />
+    <xacro:wheel.wheel
+      wheel_config="${wheel_config}"
+      wheel_separation_x="${wheel_separation_x}"
+      prefix="rr" />
     <xacro:if value="${simulation_engine == 'gazebo-classic'}">
       <gazebo>
           <plugin name="joint_states" filename="libgazebo_ros_joint_state_publisher.so">
-          <joint_name>front_left_wheel_joint</joint_name>
-          <joint_name>front_right_wheel_joint</joint_name>
-          <joint_name>rear_left_wheel_joint</joint_name>
-          <joint_name>rear_right_wheel_joint</joint_name>
+          <joint_name>fl_joint</joint_name>
+          <joint_name>fr_joint</joint_name>
+          <joint_name>rl_joint</joint_name>
+          <joint_name>rr_joint</joint_name>
         </plugin>
       </gazebo>
-      <xacro:if value="${wheel_props['wheels']['kinematics'] == 'differential'}">
+      <xacro:if value="${wheel_config['kinematics'] == 'differential'}">
         <gazebo>
           <plugin name='skid_steer_drive' filename='libgazebo_ros_diff_drive.so'>
@@ -53,17 +67,17 @@
             <update_rate>10</update_rate>
             <num_wheel_pairs>2</num_wheel_pairs>
-            <left_joint>front_left_wheel_joint</left_joint>
-            <right_joint>front_right_wheel_joint</right_joint>
-            <left_joint>rear_left_wheel_joint</left_joint>
-            <right_joint>rear_right_wheel_joint</right_joint>
-            <wheel_separation>${wheel_props['wheels']['wheel_separation']}</wheel_separation>
-            <wheel_separation>${wheel_props['wheels']['wheel_separation']}</wheel_separation>
-            <wheel_diameter>${wheel_props['wheels']['diameter']}</wheel_diameter>
-            <wheel_diameter>${wheel_props['wheels']['diameter']}</wheel_diameter>
+            <left_joint>fl_joint</left_joint>
+            <right_joint>fr_joint</right_joint>
+            <left_joint>rl_joint</left_joint>
+            <right_joint>rr_joint</right_joint>
+            <wheel_separation>${wheel_config['wheel_separation']}</wheel_separation>
+            <wheel_separation>${wheel_config['wheel_separation']}</wheel_separation>
+            <wheel_diameter>${wheel_config['wheel_radius']*2.0}</wheel_diameter>
+            <wheel_diameter>${wheel_config['wheel_radius']*2.0}</wheel_diameter>
             <max_wheel_torque>34.5</max_wheel_torque>
             <max_wheel_acceleration>2.0</max_wheel_acceleration>
             <publish_odom>true</publish_odom>
             <publish_odom_tf>true</publish_odom_tf>
-            <publish_wheel_tf>true</publish_wheel_tf>
+            <publish_wheel_tf>false</publish_wheel_tf>
             <odometry_frame>odom</odometry_frame>
             <robot_base_frame>base_link</robot_base_frame>
@@ -71,5 +85,5 @@
         </gazebo>
       </xacro:if>
-      <xacro:if value="${wheel_props['wheels']['kinematics'] == 'mecanum'}">
+      <xacro:if value="${wheel_config['kinematics'] == 'mecanum'}">
         <gazebo>
           <plugin name="object_controller" filename="libgazebo_ros_planar_move.so">

File: urdf/wheel.urdf.xacro (robot description, xacro)
@@ -2,39 +2,29 @@
 <robot xmlns:xacro="http://www.ros.org/wiki/xacro">
   <!-- wheel defining macro -->
-  <xacro:macro name="wheel" params="wheel_props prefix">
-    <xacro:property name="wheel_separation_x" value="0.44" />
-    <xacro:property name="rpy" value="0 0 0" />
-    <xacro:if value="${prefix == 'front_left'}">
+  <xacro:macro name="wheel" params="wheel_config prefix wheel_separation_x">
+    <xacro:if value="${prefix == 'fl'}">
       <xacro:property name="x" value="${wheel_separation_x/2.0}" />
-      <xacro:property name="y" value="${wheel_props['wheel_separation']/2.0}" />
-      <xacro:property name="inertia_y_offset" value="${wheel_props['inertia_y_offset']}" />
-      <xacro:property name="mesh"
-        value="file://$(find ${wheel_props['mesh_package']})/${wheel_props['folder_path']}/wheel_a.dae" />
+      <xacro:property name="y" value="${wheel_config['wheel_separation']/2.0}" />
+      <xacro:property name="inertia_y_offset" value="${wheel_config['inertia_y_offset']}" />
     </xacro:if>
-    <xacro:if value="${prefix == 'front_right'}">
+    <xacro:if value="${prefix == 'fr'}">
       <xacro:property name="x" value="${wheel_separation_x/2.0}" />
-      <xacro:property name="y" value="-${wheel_props['wheel_separation']/2.0}" />
-      <xacro:property name="inertia_y_offset" value="${-wheel_props['inertia_y_offset']}" />
-      <xacro:property name="mesh"
-        value="file://$(find ${wheel_props['mesh_package']})/${wheel_props['folder_path']}/wheel_b.dae" />
+      <xacro:property name="y" value="-${wheel_config['wheel_separation']/2.0}" />
+      <xacro:property name="inertia_y_offset" value="${-wheel_config['inertia_y_offset']}" />
     </xacro:if>
-    <xacro:if value="${prefix == 'rear_left'}">
+    <xacro:if value="${prefix == 'rl'}">
       <xacro:property name="x" value="-${wheel_separation_x/2.0}" />
-      <xacro:property name="y" value="${wheel_props['wheel_separation']/2.0}" />
-      <xacro:property name="inertia_y_offset" value="${wheel_props['inertia_y_offset']}" />
-      <xacro:property name="mesh"
-        value="file://$(find ${wheel_props['mesh_package']})/${wheel_props['folder_path']}/wheel_c.dae" />
+      <xacro:property name="y" value="${wheel_config['wheel_separation']/2.0}" />
+      <xacro:property name="inertia_y_offset" value="${wheel_config['inertia_y_offset']}" />
     </xacro:if>
-    <xacro:if value="${prefix == 'rear_right'}">
+    <xacro:if value="${prefix == 'rr'}">
       <xacro:property name="x" value="-${wheel_separation_x/2.0}" />
-      <xacro:property name="y" value="-${wheel_props['wheel_separation']/2.0}" />
-      <xacro:property name="inertia_y_offset" value="${-wheel_props['inertia_y_offset']}" />
-      <xacro:property name="mesh"
-        value="file://$(find ${wheel_props['mesh_package']})/${wheel_props['folder_path']}/wheel_d.dae" />
+      <xacro:property name="y" value="-${wheel_config['wheel_separation']/2.0}" />
+      <xacro:property name="inertia_y_offset" value="${-wheel_config['inertia_y_offset']}" />
     </xacro:if>
     <link name="${prefix}_wheel_link">
        <visual>
         <geometry>
-            <mesh filename="${mesh}" scale="1.0 1.0 1.0" />
+            <mesh filename="file://$(find ${wheel_config['mesh_package']})/${wheel_config['folder_path']}/${prefix}_wheel.dae" />
         </geometry>
         <origin xyz="0.0 0.0 0.0" rpy="0.0 0.0 0.0" />
@@ -42,5 +32,5 @@
       <collision>
         <geometry>
-            <mesh filename="file://$(find ${wheel_props['mesh_package']})/${wheel_props['folder_path']}/collision.stl" scale="1.0 1.0 1.0" />
+            <mesh filename="file://$(find ${wheel_config['mesh_package']})/${wheel_config['folder_path']}/collision.stl" />
         </geometry>
         <origin xyz="0.0 0.0 0.0" rpy="0.0 0.0 0.0" />
@@ -48,14 +38,14 @@
       <inertial>
         <origin xyz="0.0 ${inertia_y_offset} 0.0" rpy="0.0 0.0 0.0"/>
-        <mass value="${wheel_props['mass']}" />
-        <inertia ixx="${wheel_props['inertia']['ixx']}"
+        <mass value="${wheel_config['mass']}" />
+        <inertia ixx="${wheel_config['inertia']['ixx']}"
                  ixy="0.0"
                  ixz="0.0"
-                 iyy="${wheel_props['inertia']['iyy']}"
+                 iyy="${wheel_config['inertia']['iyy']}"
                  iyz="0.0"
-                 izz="${wheel_props['inertia']['izz']}" />
+                 izz="${wheel_config['inertia']['izz']}" />
       </inertial>
     </link>
-    <joint name="${prefix}_wheel_joint" type="continuous">
+    <joint name="${prefix}_joint" type="continuous">
       <parent link="body_link" />
       <child link="${prefix}_wheel_link" />
