Commit message: Update readme, GPS antenna and joint-link order

File: urdf/body.urdf.xacro (robot description, xacro)
@@ -28,8 +28,4 @@
       </inertial>
     </link>
-    <link name="imu_link"></link>
-    <link name="front_light_link"></link>
-    <link name="rear_light_link"></link>
-    <link name="cover_link"></link>
     <joint name="base_link_to_body_link_joint" type="fixed">
       <origin xyz="0.0 0.0 ${wheel_radius}" rpy="0.0 0.0 0.0" />
@@ -37,4 +33,5 @@
       <child link="body_link" />
     </joint>
+    <link name="imu_link"></link>
     <joint name="body_link_to_imu_link_joint" type="fixed">
       <origin xyz="${imu_pos_x} ${imu_pos_y} ${imu_pos_z}"
@@ -43,4 +40,5 @@
       <child link="imu_link" />
     </joint>
+    <link name="front_light_link"></link>
     <joint name="body_link_front_light_link_joint" type="fixed">
       <origin xyz="0.362 0.0 0.0" rpy="0.0 0.0 0.0" />
@@ -48,4 +46,5 @@
       <child link="front_light_link" />
     </joint>
+    <link name="rear_light_link"></link>
     <joint name="body_link_to_rear_light_link_joint" type="fixed">
       <origin xyz="-0.362 0.0 0.0" rpy="0.0 0.0 ${pi}" />
@@ -53,4 +52,5 @@
       <child link="rear_light_link" />
     </joint>
+    <link name="cover_link"></link>
     <joint name="body_link_to_cover_link_joint" type="fixed">
       <origin xyz="0.0 0.0 0.1715" rpy="0.0 0.0 0.0" />

File: urdf/components/external_antenna.urdf.xacro (robot description, xacro)
@@ -6,4 +6,7 @@
                        topic:=gps
                        frame_id:=gps
+                       initial_latitude:=53.1978
+                       initial_longitude:=18.3735
+                       initial_altitude:=89.0
                        simulation_engine:=gazebo-classic">
     <xacro:if value="${tf_prefix == 'None'}">
@@ -39,5 +42,5 @@
     <link name="${tf_prefix_ext}${frame_id}"></link>
     <joint name="${tf_prefix_ext}external_antenna_link_to_${tf_prefix_ext}${frame_id}_joint" type="fixed">
-      <origin xyz="0.0 0.0 0.0" rpy="0.0 0.0 0.0" />
+      <origin xyz="0.045 0.0 0.004" rpy="0.0 0.0 0.0" />
       <parent link="${tf_prefix_ext}external_antenna_link" />
       <child link="${tf_prefix_ext}${frame_id}" />
@@ -45,5 +48,5 @@
     <!-- based on Teltonika RUTX11 datasheet and measuremets-->
     <gazebo>
-      <plugin name="gps_controller" filename="libhector_gazebo_ros_gps.so">
+      <plugin name="gps" filename="libhector_gazebo_ros_gps.so">
         <updateRate>5</updateRate>
         <robotNamespace>/</robotNamespace>
@@ -52,8 +55,8 @@
         <topicName>/${topic}/fix</topicName>
         <velocityTopicName>/${topic}/vel</velocityTopicName>
-        <referenceLatitude>53.1978</referenceLatitude>
-        <referenceLongitude>18.3735</referenceLongitude>
-        <referenceHeading>0</referenceHeading>
-        <referenceAltitude>0</referenceAltitude>
+        <referenceLatitude>${initial_latitude}</referenceLatitude>
+        <referenceLongitude>${initial_longitude}</referenceLongitude>
+        <referenceHeading>0.0</referenceHeading>
+        <referenceAltitude>${initial_altitude}</referenceAltitude>
         <drift>0.0001 0.0001 0.0001</drift>
         <gaussianNoise>3.0 3.0 3.0</gaussianNoise>

File: urdf/panther.urdf.xacro (robot description, xacro)
@@ -24,5 +24,5 @@
     wheel_config_path="$(arg wheel_config_path)"
     simulation_engine="$(arg simulation_engine)" />
-  <!-- <xacro:include filename="$(find ros_components_description)/urdf/rplidar_s1.gazebo.xacro" ns="lidar" />
+  <xacro:include filename="$(find ros_components_description)/urdf/rplidar_s1.gazebo.xacro" ns="lidar" />
   <xacro:lidar.rplidar_s1
     parent_link="cover_link"
@@ -30,9 +30,4 @@
     rpy="0.0 0.0 0.0"
     use_gpu="$(arg use_gpu)"
-    simulation_engine="$(arg simulation_engine)" /> -->
-  <xacro:include filename="$(find panther_description)/urdf/components/external_antenna.urdf.xacro" ns="antenna" />
-  <xacro:antenna.external_antenna
-    parent_link="cover_link"
-    xyz="0.0 0.0 0.0"
-    rpy="0.0 0.0 0.0" />
+    simulation_engine="$(arg simulation_engine)" />
 </robot>

Commit message: Change order of links and joints

File: urdf/body.urdf.xacro (robot description, xacro)
@@ -7,4 +7,9 @@
     imu_rot_r imu_rot_p imu_rot_y" >
     <link name="base_link"></link>
+    <joint name="base_link_to_body_link_joint" type="fixed">
+      <origin xyz="0.0 0.0 ${wheel_radius}" rpy="0.0 0.0 0.0" />
+      <parent link="base_link" />
+      <child link="body_link" />
+    </joint>
     <link name="body_link">
       <visual>
@@ -28,10 +33,4 @@
       </inertial>
     </link>
-    <joint name="base_link_to_body_link_joint" type="fixed">
-      <origin xyz="0.0 0.0 ${wheel_radius}" rpy="0.0 0.0 0.0" />
-      <parent link="base_link" />
-      <child link="body_link" />
-    </joint>
-    <link name="imu_link"></link>
     <joint name="body_link_to_imu_link_joint" type="fixed">
       <origin xyz="${imu_pos_x} ${imu_pos_y} ${imu_pos_z}"
@@ -40,5 +39,5 @@
       <child link="imu_link" />
     </joint>
-    <link name="front_light_link"></link>
+    <link name="imu_link"></link>
     <joint name="body_link_front_light_link_joint" type="fixed">
       <origin xyz="0.362 0.0 0.0" rpy="0.0 0.0 0.0" />
@@ -46,5 +45,5 @@
       <child link="front_light_link" />
     </joint>
-    <link name="rear_light_link"></link>
+    <link name="front_light_link"></link>
     <joint name="body_link_to_rear_light_link_joint" type="fixed">
       <origin xyz="-0.362 0.0 0.0" rpy="0.0 0.0 ${pi}" />
@@ -52,5 +51,5 @@
       <child link="rear_light_link" />
     </joint>
-    <link name="cover_link"></link>
+    <link name="rear_light_link"></link>
     <joint name="body_link_to_cover_link_joint" type="fixed">
       <origin xyz="0.0 0.0 0.1715" rpy="0.0 0.0 0.0" />
@@ -58,4 +57,5 @@
       <child link="cover_link" />
     </joint>
+    <link name="cover_link"></link>
     <xacro:if value="${simulation_engine == 'gazebo-classic'}">
       <!-- based on PhidgetSpatial datasheet -->

File: urdf/components/external_antenna.urdf.xacro (robot description, xacro)
@@ -16,4 +16,9 @@
       <xacro:property name="tf_prefix_ext" value="${tf_prefix}_" />
     </xacro:unless>
+    <joint name="${parent_link}_to_${tf_prefix_ext}external_antenna_link_joint" type="fixed">
+      <origin xyz="${xyz}" rpy="${rpy}" />
+      <parent link="${parent_link}" />
+      <child link="${tf_prefix_ext}external_antenna_link" />
+    </joint>
     <link name="${tf_prefix_ext}external_antenna_link">
       <visual>
@@ -35,10 +40,4 @@
       </inertial>
     </link>
-    <joint name="${parent_link}_to_${tf_prefix_ext}external_antenna_link_joint" type="fixed">
-      <origin xyz="${xyz}" rpy="${rpy}" />
-      <parent link="${parent_link}" />
-      <child link="${tf_prefix_ext}external_antenna_link" />
-    </joint>
-    <link name="${tf_prefix_ext}${frame_id}"></link>
     <joint name="${tf_prefix_ext}external_antenna_link_to_${tf_prefix_ext}${frame_id}_joint" type="fixed">
       <origin xyz="0.045 0.0 0.004" rpy="0.0 0.0 0.0" />
@@ -46,4 +45,5 @@
       <child link="${tf_prefix_ext}${frame_id}" />
     </joint>
+    <link name="${tf_prefix_ext}${frame_id}"></link>
     <!-- based on Teltonika RUTX11 datasheet and measuremets-->
     <gazebo>

File: urdf/wheel.urdf.xacro (robot description, xacro)
@@ -23,4 +23,14 @@
       <xacro:property name="inertia_y_offset" value="${-wheel_config['inertia_y_offset']}" />
     </xacro:if>
+    <joint name="${prefix}_joint" type="continuous">
+      <parent link="body_link" />
+      <child link="${prefix}_wheel_link" />
+      <origin xyz="${x} ${y} 0.0" rpy="0.0 0.0 0.0" />
+      <axis xyz="0.0 1.0 0.0" />
+      <limit effort="34.5"
+             velocity="2.0" />
+      <dynamics damping="0.01"
+                friction="0.01"/>
+    </joint>
     <link name="${prefix}_wheel_link">
        <visual>
@@ -47,14 +57,4 @@
       </inertial>
     </link>
-    <joint name="${prefix}_joint" type="continuous">
-      <parent link="body_link" />
-      <child link="${prefix}_wheel_link" />
-      <origin xyz="${x} ${y} 0.0" rpy="0.0 0.0 0.0" />
-      <axis xyz="0.0 1.0 0.0" />
-      <limit effort="34.5"
-             velocity="2.0" />
-      <dynamics damping="0.01"
-                friction="0.01"/>
-    </joint>
   </xacro:macro>
 </robot>

Commit message: Update urdf/body.urdf.xacro
Co-authored-by: Maciej Stępień <maciek1284@outlook.com>

File: urdf/body.urdf.xacro (robot description, xacro)
@@ -6,5 +6,5 @@
     imu_pos_x imu_pos_y imu_pos_z
     imu_rot_r imu_rot_p imu_rot_y" >
-    <link name="base_link"></link>
+    <link name="base_link" />
     <joint name="base_link_to_body_link_joint" type="fixed">
       <origin xyz="0.0 0.0 ${wheel_radius}" rpy="0.0 0.0 0.0" />

Commit message: Addvreview changes

File: urdf/body.urdf.xacro (robot description, xacro)
@@ -39,5 +39,5 @@
       <child link="imu_link" />
     </joint>
-    <link name="imu_link"></link>
+    <link name="imu_link" />
     <joint name="body_link_front_light_link_joint" type="fixed">
       <origin xyz="0.362 0.0 0.0" rpy="0.0 0.0 0.0" />
@@ -45,5 +45,5 @@
       <child link="front_light_link" />
     </joint>
-    <link name="front_light_link"></link>
+    <link name="front_light_link" />
     <joint name="body_link_to_rear_light_link_joint" type="fixed">
       <origin xyz="-0.362 0.0 0.0" rpy="0.0 0.0 ${pi}" />
@@ -51,5 +51,5 @@
       <child link="rear_light_link" />
     </joint>
-    <link name="rear_light_link"></link>
+    <link name="rear_light_link" />
     <joint name="body_link_to_cover_link_joint" type="fixed">
       <origin xyz="0.0 0.0 0.1715" rpy="0.0 0.0 0.0" />
@@ -57,5 +57,5 @@
       <child link="cover_link" />
     </joint>
-    <link name="cover_link"></link>
+    <link name="cover_link" />
     <xacro:if value="${simulation_engine == 'gazebo-classic'}">
       <!-- based on PhidgetSpatial datasheet -->

File: urdf/components/external_antenna.urdf.xacro (robot description, xacro)
@@ -45,5 +45,5 @@
       <child link="${tf_prefix_ext}${frame_id}" />
     </joint>
-    <link name="${tf_prefix_ext}${frame_id}"></link>
+    <link name="${tf_prefix_ext}${frame_id}" />
     <!-- based on Teltonika RUTX11 datasheet and measuremets-->
     <gazebo>

File: urdf/panther_macro.urdf.xacro (robot description, xacro)
@@ -65,8 +65,8 @@
             <wheelDiameter>${wheel_config['wheel_radius']*2.0}</wheelDiameter>
             <torque>34.5</torque>
-            <leftFrontJoint>fl_joint</leftFrontJoint>
-            <rightFrontJoint>fr_joint</rightFrontJoint>
-            <leftRearJoint>rl_joint</leftRearJoint>
-            <rightRearJoint>rr_joint</rightRearJoint>
+            <leftFrontJoint>fl_wheel_joint</leftFrontJoint>
+            <rightFrontJoint>fr_wheel_joint</rightFrontJoint>
+            <leftRearJoint>rl_wheel_joint</leftRearJoint>
+            <rightRearJoint>rr_wheel_joint</rightRearJoint>
             <topicName>cmd_vel</topicName>
             <commandTopic>cmd_vel</commandTopic>

File: urdf/wheel.urdf.xacro (robot description, xacro)
@@ -23,5 +23,5 @@
       <xacro:property name="inertia_y_offset" value="${-wheel_config['inertia_y_offset']}" />
     </xacro:if>
-    <joint name="${prefix}_joint" type="continuous">
+    <joint name="${prefix}_wheel_joint" type="continuous">
       <parent link="body_link" />
       <child link="${prefix}_wheel_link" />
@@ -55,15 +55,15 @@
       </inertial>
     </link>
-    <transmission name="${prefix}_transmission" type="SimpleTransmission">
+    <transmission name="${prefix}_wheel_transmission" type="SimpleTransmission">
       <type>transmission_interface/SimpleTransmission</type>
-      <joint name="${prefix}_joint">
+      <joint name="${prefix}_wheel_joint">
         <hardwareInterface>hardware_interface/EffortJointInterface</hardwareInterface>
       </joint>
-      <actuator name="${prefix}_actuator">
+      <actuator name="${prefix}_wheel_actuator">
         <mechanicalReduction>1</mechanicalReduction>
         <hardwareInterface>hardware_interface/EffortJointInterface</hardwareInterface>
       </actuator>
     </transmission>
-    <gazebo reference="${prefix}_joint">
+    <gazebo reference="${prefix}_wheel_joint">
       <provideFeedback>true</provideFeedback>
     </gazebo>

Commit message: Fix ros1 branch differences

File: urdf/body.urdf.xacro (robot description, xacro)
@@ -6,5 +6,5 @@
     imu_pos_x imu_pos_y imu_pos_z
     imu_rot_r imu_rot_p imu_rot_y" >
-    <link name="base_link"></link>
+    <link name="base_link" />
     <joint name="base_link_to_body_link_joint" type="fixed">
       <origin xyz="0.0 0.0 ${wheel_radius}" rpy="0.0 0.0 0.0" />
@@ -39,5 +39,5 @@
       <child link="imu_link" />
     </joint>
-    <link name="imu_link"></link>
+    <link name="imu_link" />
     <joint name="body_link_front_light_link_joint" type="fixed">
       <origin xyz="0.362 0.0 0.0" rpy="0.0 0.0 0.0" />
@@ -45,5 +45,5 @@
       <child link="front_light_link" />
     </joint>
-    <link name="front_light_link"></link>
+    <link name="front_light_link" />
     <joint name="body_link_to_rear_light_link_joint" type="fixed">
       <origin xyz="-0.362 0.0 0.0" rpy="0.0 0.0 ${pi}" />
@@ -51,5 +51,5 @@
       <child link="rear_light_link" />
     </joint>
-    <link name="rear_light_link"></link>
+    <link name="rear_light_link" />
     <joint name="body_link_to_cover_link_joint" type="fixed">
       <origin xyz="0.0 0.0 0.1715" rpy="0.0 0.0 0.0" />
@@ -57,5 +57,5 @@
       <child link="cover_link" />
     </joint>
-    <link name="cover_link"></link>
+    <link name="cover_link" />
     <xacro:if value="${simulation_engine == 'gazebo-classic'}">
       <!-- based on PhidgetSpatial datasheet -->
@@ -76,5 +76,5 @@
         </plugin>
       </gazebo>
-  </xacro:if>
+    </xacro:if>
   </xacro:macro>
 </robot>

File: urdf/panther_macro.urdf.xacro (robot description, xacro)
@@ -54,8 +54,8 @@
       <gazebo>
           <plugin name="joint_states" filename="libgazebo_ros_joint_state_publisher.so">
-          <joint_name>fl_joint</joint_name>
-          <joint_name>fr_joint</joint_name>
-          <joint_name>rl_joint</joint_name>
-          <joint_name>rr_joint</joint_name>
+          <joint_name>fl_wheel_joint</joint_name>
+          <joint_name>fr_wheel_joint</joint_name>
+          <joint_name>rl_wheel_joint</joint_name>
+          <joint_name>rr_wheel_joint</joint_name>
         </plugin>
       </gazebo>
@@ -67,8 +67,8 @@
             <update_rate>10</update_rate>
             <num_wheel_pairs>2</num_wheel_pairs>
-            <left_joint>fl_joint</left_joint>
-            <right_joint>fr_joint</right_joint>
-            <left_joint>rl_joint</left_joint>
-            <right_joint>rr_joint</right_joint>
+            <left_joint>fl_wheel_joint</left_joint>
+            <right_joint>fr_wheel_joint</right_joint>
+            <left_joint>rl_wheel_joint</left_joint>
+            <right_joint>rr_wheel_joint</right_joint>
             <wheel_separation>${wheel_config['wheel_separation']}</wheel_separation>
             <wheel_separation>${wheel_config['wheel_separation']}</wheel_separation>
@@ -102,5 +102,5 @@
         </gazebo>
       </xacro:if>
-  </xacro:if>
+    </xacro:if>
   </xacro:macro>
 </robot>

File: urdf/wheel.urdf.xacro (robot description, xacro)
@@ -23,18 +23,16 @@
       <xacro:property name="inertia_y_offset" value="${-wheel_config['inertia_y_offset']}" />
     </xacro:if>
-    <joint name="${prefix}_joint" type="continuous">
+    <joint name="${prefix}_wheel_joint" type="continuous">
       <parent link="body_link" />
       <child link="${prefix}_wheel_link" />
       <origin xyz="${x} ${y} 0.0" rpy="0.0 0.0 0.0" />
       <axis xyz="0.0 1.0 0.0" />
-      <limit effort="34.5"
-             velocity="2.0" />
-      <dynamics damping="0.01"
-                friction="0.01"/>
+      <limit effort="34.5" velocity="2.0" />
+      <dynamics damping="0.01" friction="0.01" />
     </joint>
     <link name="${prefix}_wheel_link">
        <visual>
         <geometry>
-            <mesh filename="file://$(find ${wheel_config['mesh_package']})/${wheel_config['folder_path']}/${prefix}_wheel.dae" />
+          <mesh filename="file://$(find ${wheel_config['mesh_package']})/${wheel_config['folder_path']}/${prefix}_wheel.dae" />
         </geometry>
         <origin xyz="0.0 0.0 0.0" rpy="0.0 0.0 0.0" />
@@ -42,5 +40,5 @@
       <collision>
         <geometry>
-            <mesh filename="file://$(find ${wheel_config['mesh_package']})/${wheel_config['folder_path']}/collision.stl" />
+          <mesh filename="file://$(find ${wheel_config['mesh_package']})/${wheel_config['folder_path']}/collision.stl" />
         </geometry>
         <origin xyz="0.0 0.0 0.0" rpy="0.0 0.0 0.0" />
@@ -57,4 +55,11 @@
       </inertial>
     </link>
+    <gazebo reference="${prefix}_wheel_link">
+      <mu1 value="0.85"/>
+			<mu2 value="0.85"/>
+			<kp value="100000000.0" />
+			<kd value="5.0" />
+			<fdir1 value="1 0 0"/>
+    </gazebo>
   </xacro:macro>
 </robot>

Commit message: Update to URDF guide

File: urdf/body.urdf.xacro (robot description, xacro)
@@ -7,5 +7,5 @@
     imu_rot_r imu_rot_p imu_rot_y" >
     <link name="base_link" />
-    <joint name="base_link_to_body_link_joint" type="fixed">
+    <joint name="base_to_body_joint" type="fixed">
       <origin xyz="0.0 0.0 ${wheel_radius}" rpy="0.0 0.0 0.0" />
       <parent link="base_link" />
@@ -14,17 +14,17 @@
     <link name="body_link">
       <visual>
+        <origin xyz="0.0 0.0 0.0" rpy="0.0 0.0 0.0"/>
         <geometry>
           <mesh filename="file://$(find panther_description)/meshes/body.dae" />
         </geometry>
-        <origin xyz="0.0 0.0 0.0" rpy="0.0 0.0 0.0"/>
       </visual>
       <collision>
+        <origin xyz="0.0 0.0 0.0" rpy="0.0 0.0 0.0"/>
         <geometry>
           <mesh filename="file://$(find panther_description)/meshes/body_collision.stl" />
         </geometry>
-        <origin xyz="0.0 0.0 0.0" rpy="0.0 0.0 0.0"/>
       </collision>
       <inertial>
-        <origin xyz="-0.008 0.01 0.029" rpy="0.0 0.0 0.0"/>
+        <origin xyz="0.0 0.0 0.0" rpy="0.0 0.0 0.0" />
         <mass value="43.0" />
         <inertia ixx="2.630036" ixy="-0.023480" ixz="0.052320"
@@ -33,5 +33,5 @@
       </inertial>
     </link>
-    <joint name="body_link_to_imu_link_joint" type="fixed">
+    <joint name="body_to_imu_joint" type="fixed">
       <origin xyz="${imu_pos_x} ${imu_pos_y} ${imu_pos_z}"
               rpy="${imu_rot_r} ${imu_rot_p} ${imu_rot_y}" />
@@ -40,5 +40,5 @@
     </joint>
     <link name="imu_link" />
-    <joint name="body_link_front_light_link_joint" type="fixed">
+    <joint name="body_front_light_joint" type="fixed">
       <origin xyz="0.362 0.0 0.0" rpy="0.0 0.0 0.0" />
       <parent link="body_link" />
@@ -46,5 +46,5 @@
     </joint>
     <link name="front_light_link" />
-    <joint name="body_link_to_rear_light_link_joint" type="fixed">
+    <joint name="body_to_rear_light_joint" type="fixed">
       <origin xyz="-0.362 0.0 0.0" rpy="0.0 0.0 ${pi}" />
       <parent link="body_link" />
@@ -52,5 +52,5 @@
     </joint>
     <link name="rear_light_link" />
-    <joint name="body_link_to_cover_link_joint" type="fixed">
+    <joint name="body_to_cover_joint" type="fixed">
       <origin xyz="0.0 0.0 0.1715" rpy="0.0 0.0 0.0" />
       <parent link="body_link" />

File: urdf/components/external_antenna.urdf.xacro (robot description, xacro)
@@ -16,5 +16,5 @@
       <xacro:property name="tf_prefix_ext" value="${tf_prefix}_" />
     </xacro:unless>
-    <joint name="${parent_link}_to_${tf_prefix_ext}external_antenna_link_joint" type="fixed">
+    <joint name="${parent_link.rstrip('_link')}_to_${tf_prefix_ext}external_antenna_joint" type="fixed">
       <origin xyz="${xyz}" rpy="${rpy}" />
       <parent link="${parent_link}" />
@@ -23,22 +23,22 @@
     <link name="${tf_prefix_ext}external_antenna_link">
       <visual>
+        <origin xyz="0.0 0.0 0.0" rpy="0.0 0.0 0.0"/>
         <geometry>
           <mesh filename="file://$(find panther_description)/meshes/components/external_antenna.dae" />
         </geometry>
-        <origin xyz="0.0 0.0 0.0" rpy="0.0 0.0 0.0"/>
       </visual>
       <collision>
+        <origin xyz="0.0 0.0 0.0" rpy="0.0 0.0 0.0"/>
         <geometry>
           <mesh filename="file://$(find panther_description)/meshes/components/external_antenna_collision.stl" />
         </geometry>
-        <origin xyz="0.0 0.0 0.0" rpy="0.0 0.0 0.0"/>
       </collision>
       <inertial>
+        <origin xyz="0.045 0.0 0.0058" rpy="0.0 0.0 0.0"/>
         <mass value="0.59" />
         <inertia ixx="0.003964" ixy="0.0" ixz="0.0" iyy="0.0003964" iyz="0.0" izz="0.0004177" />
-        <origin xyz="0.045 0.0 0.0058" rpy="0.0 0.0 0.0"/>
       </inertial>
     </link>
-    <joint name="${tf_prefix_ext}external_antenna_link_to_${tf_prefix_ext}${frame_id}_joint" type="fixed">
+    <joint name="${tf_prefix_ext}external_antenna_to_${tf_prefix_ext}${frame_id.rstrip('_link')}_joint" type="fixed">
       <origin xyz="0.045 0.0 0.0058" rpy="0.0 0.0 0.0" />
       <parent link="${tf_prefix_ext}external_antenna_link" />

File: urdf/wheel.urdf.xacro (robot description, xacro)
@@ -24,7 +24,7 @@
     </xacro:if>
     <joint name="${prefix}_wheel_joint" type="continuous">
+      <origin xyz="${x} ${y} 0.0" rpy="0.0 0.0 0.0" />
       <parent link="body_link" />
       <child link="${prefix}_wheel_link" />
-      <origin xyz="${x} ${y} 0.0" rpy="0.0 0.0 0.0" />
       <axis xyz="0.0 1.0 0.0" />
       <limit effort="34.5" velocity="2.0" />
@@ -32,18 +32,18 @@
     </joint>
     <link name="${prefix}_wheel_link">
-       <visual>
+      <visual>
+        <origin xyz="0.0 0.0 0.0" rpy="0.0 0.0 0.0" />
         <geometry>
           <mesh filename="file://$(find ${wheel_config['mesh_package']})/${wheel_config['folder_path']}/${prefix}_wheel.dae" />
         </geometry>
-        <origin xyz="0.0 0.0 0.0" rpy="0.0 0.0 0.0" />
       </visual>
       <collision>
+        <origin xyz="0.0 0.0 0.0" rpy="0.0 0.0 0.0" />
         <geometry>
-          <mesh filename="file://$(find ${wheel_config['mesh_package']})/${wheel_config['folder_path']}/collision.stl" />
+          <mesh filename="file://$(find ${wheel_config['mesh_package']})/${wheel_config['folder_path']}/wheel_collision.stl" />
         </geometry>
-        <origin xyz="0.0 0.0 0.0" rpy="0.0 0.0 0.0" />
       </collision>
       <inertial>
-        <origin xyz="0.0 ${inertia_y_offset} 0.0" rpy="0.0 0.0 0.0"/>
+        <origin xyz="0.0 ${inertia_y_offset} 0.0" rpy="0.0 0.0 0.0" />
         <mass value="${wheel_config['mass']}" />
         <inertia ixx="${wheel_config['inertia']['ixx']}"
@@ -55,11 +55,4 @@
       </inertial>
     </link>
-    <gazebo reference="${prefix}_wheel_link">
-      <mu1 value="0.85" />
-      <mu2 value="0.85" />
-      <kp value="100000000.0" />
-      <kd value="5.0" />
-      <fdir1 value="1.0 0.0 0.0" />
-    </gazebo>
   </xacro:macro>
 </robot>
