Commit message: FIx joint name typo

File: urdf/body.urdf.xacro (robot description, xacro)
@@ -40,5 +40,5 @@
     </joint>
     <link name="imu_link" />
-    <joint name="body_front_light_joint" type="fixed">
+    <joint name="body_to_front_light_joint" type="fixed">
       <origin xyz="0.362 0.0 0.0" rpy="0.0 0.0 0.0" />
       <parent link="body_link" />

Commit message: Last update

File: urdf/body.urdf.xacro (robot description, xacro)
@@ -7,5 +7,5 @@
     imu_rot_r imu_rot_p imu_rot_y" >
     <link name="base_link" />
-    <joint name="base_link_to_body_link_joint" type="fixed">
+    <joint name="base_to_body_joint" type="fixed">
       <origin xyz="0.0 0.0 ${wheel_radius}" rpy="0.0 0.0 0.0" />
       <parent link="base_link" />
@@ -14,17 +14,17 @@
     <link name="body_link">
       <visual>
+        <origin xyz="0.0 0.0 0.0" rpy="0.0 0.0 0.0"/>
         <geometry>
           <mesh filename="file://$(find panther_description)/meshes/body.dae" />
         </geometry>
-        <origin xyz="0.0 0.0 0.0" rpy="0.0 0.0 0.0"/>
       </visual>
       <collision>
+        <origin xyz="0.0 0.0 0.0" rpy="0.0 0.0 0.0"/>
         <geometry>
           <mesh filename="file://$(find panther_description)/meshes/body_collision.stl" />
         </geometry>
-        <origin xyz="0.0 0.0 0.0" rpy="0.0 0.0 0.0"/>
       </collision>
       <inertial>
-        <origin xyz="-0.008 0.01 0.029" rpy="0.0 0.0 0.0"/>
+        <origin xyz="0.0 0.0 0.0" rpy="0.0 0.0 0.0" />
         <mass value="43.0" />
         <inertia ixx="2.630036" ixy="-0.023480" ixz="0.052320"
@@ -33,5 +33,5 @@
       </inertial>
     </link>
-    <joint name="body_link_to_imu_link_joint" type="fixed">
+    <joint name="body_to_imu_joint" type="fixed">
       <origin xyz="${imu_pos_x} ${imu_pos_y} ${imu_pos_z}"
               rpy="${imu_rot_r} ${imu_rot_p} ${imu_rot_y}" />
@@ -40,5 +40,5 @@
     </joint>
     <link name="imu_link" />
-    <joint name="body_link_front_light_link_joint" type="fixed">
+    <joint name="body_to_front_light_joint" type="fixed">
       <origin xyz="0.362 0.0 0.0" rpy="0.0 0.0 0.0" />
       <parent link="body_link" />
@@ -46,5 +46,5 @@
     </joint>
     <link name="front_light_link" />
-    <joint name="body_link_to_rear_light_link_joint" type="fixed">
+    <joint name="body_to_rear_light_joint" type="fixed">
       <origin xyz="-0.362 0.0 0.0" rpy="0.0 0.0 ${pi}" />
       <parent link="body_link" />
@@ -52,5 +52,5 @@
     </joint>
     <link name="rear_light_link" />
-    <joint name="body_link_to_cover_link_joint" type="fixed">
+    <joint name="body_to_cover_joint" type="fixed">
       <origin xyz="0.0 0.0 0.1715" rpy="0.0 0.0 0.0" />
       <parent link="body_link" />

File: urdf/panther_macro.urdf.xacro (robot description, xacro)
@@ -74,7 +74,7 @@
             <odometryTopic>odom</odometryTopic>
             <odometryFrame>odom</odometryFrame>
-            <covariance_x>0.000100</covariance_x>
-            <covariance_y>0.000100</covariance_y>
-            <covariance_yaw>0.010000</covariance_yaw>
+            <covariance_x>0.0001</covariance_x>
+            <covariance_y>0.0001</covariance_y>
+            <covariance_yaw>0.0100</covariance_yaw>
           </plugin>
         </gazebo>

File: urdf/wheel.urdf.xacro (robot description, xacro)
@@ -24,7 +24,7 @@
     </xacro:if>
     <joint name="${prefix}_wheel_joint" type="continuous">
+      <origin xyz="${x} ${y} 0.0" rpy="0.0 0.0 0.0" />
       <parent link="body_link" />
       <child link="${prefix}_wheel_link" />
-      <origin xyz="${x} ${y} 0.0" rpy="0.0 0.0 0.0" />
       <axis xyz="0.0 1.0 0.0" />
       <limit effort="34.5" velocity="2.0" />
@@ -32,18 +32,18 @@
     </joint>
     <link name="${prefix}_wheel_link">
-       <visual>
+      <visual>
+        <origin xyz="0.0 0.0 0.0" rpy="0.0 0.0 0.0" />
         <geometry>
-            <mesh filename="file://$(find ${wheel_config['mesh_package']})/${wheel_config['folder_path']}/${prefix}_wheel.dae" />
+          <mesh filename="file://$(find ${wheel_config['mesh_package']})/${wheel_config['folder_path']}/${prefix}_wheel.dae" />
         </geometry>
-        <origin xyz="0.0 0.0 0.0" rpy="0.0 0.0 0.0" />
       </visual>
       <collision>
+        <origin xyz="0.0 0.0 0.0" rpy="0.0 0.0 0.0" />
         <geometry>
-            <mesh filename="file://$(find ${wheel_config['mesh_package']})/${wheel_config['folder_path']}/collision.stl" />
+          <mesh filename="file://$(find ${wheel_config['mesh_package']})/${wheel_config['folder_path']}/wheel_collision.stl" />
         </geometry>
-        <origin xyz="0.0 0.0 0.0" rpy="0.0 0.0 0.0" />
       </collision>
       <inertial>
-        <origin xyz="0.0 ${inertia_y_offset} 0.0" rpy="0.0 0.0 0.0"/>
+        <origin xyz="0.0 ${inertia_y_offset} 0.0" rpy="0.0 0.0 0.0" />
         <mass value="${wheel_config['mass']}" />
         <inertia ixx="${wheel_config['inertia']['ixx']}"
@@ -68,11 +68,4 @@
       <provideFeedback>true</provideFeedback>
     </gazebo>
-    <gazebo reference="${prefix}_wheel_link">
-      <mu1 value="0.8" />
-      <mu2 value="0.8" />
-      <kp value="100000000.0" />
-      <kd value="10.0" />
-      <fdir1 value="1.0 0.0 0.0" />
-    </gazebo>
   </xacro:macro>
 </robot>
